Commit message: added gz configurations

File: install/abb_irb140_description/share/abb_irb140_description/urdf/irb140.urdf (robot description, URDF)
Before this commit: robot abb_irb140, 10 links, 9 joints
Links:
- removed link world
- link base_link: mass 26.383023 -> None
- link link_1: mass 34.629380 -> None
- link link_2: mass 16.116764 -> None
- link link_3: mass 16.752833 -> None
- link link_4: mass 3.755635 -> None
- link link_5: mass 0.307952 -> None
- link link_6: mass 0.054413 -> None
Joints:
- removed joint world-base_link
- joint joint_1: limit lower=-3.1416 upper=3.1416 effort=200 velocity=2.618 -> lower=-3.1416 upper=3.1416 effort=0 velocity=2.618
- joint joint_2: limit lower=-1.7453 upper=1.9199 effort=200 velocity=2.618 -> lower=-1.7453 upper=1.9199 effort=0 velocity=2.618
- joint joint_3: limit lower=-1.0472 upper=1.1345 effort=150 velocity=2.618 -> lower=-1.0472 upper=1.1345 effort=0 velocity=2.618
- joint joint_4: limit lower=-3.49 upper=3.49 effort=50 velocity=6.2832 -> lower=-3.49 upper=3.49 effort=0 velocity=6.2832
- joint joint_5: limit lower=-2.0944 upper=2.0944 effort=50 velocity=6.2832 -> lower=-2.0944 upper=2.0944 effort=0 velocity=6.2832
- joint joint_6: limit lower=-6.9813 upper=6.9813 effort=20 velocity=7.854 -> lower=-6.9813 upper=6.9813 effort=0 velocity=7.854
