Commit message: end effector successfully modelled

File: urdf/irb140_pneumonic_gripper.urdf (robot description, URDF)
Before this commit: robot irb140_pneumonic_gripper, 1 links, 0 joints
Links:
- added link left_gripper_link_1; collision box size=0.025 0.03 0.022; visual mesh filename=package://abb_irb140_description/meshes/abb_irb140_pneumoni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 scale=0.001 0.001 0.001
- added link left_gripper_link_2; collision box size=0.025 0.03 0.011; visual mesh filename=package://abb_irb140_description/meshes/abb_irb140_pneumoni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 scale=0.001 0.001 0.001
- added link left_gripper_link_3; collision box size=0.025 0.03 0.011; visual mesh filename=package://abb_irb140_description/meshes/abb_irb140_pneumoni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 scale=0.001 0.001 0.001
- added link left_gripper_link_4; collision box size=0.025 0.03 0.011; visual mesh filename=package://abb_irb140_description/meshes/abb_irb140_pneumoni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 scale=0.001 0.001 0.001
- added link left_gripper_link_5; collision box size=0.025 0.03 0.011; visual mesh filename=package://abb_irb140_description/meshes/abb_irb140_pneumoni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 scale=0.001 0.001 0.001
- added link left_gripper_link_6; collision box size=0.025 0.03 0.011; visual mesh filename=package://abb_irb140_description/meshes/abb_irb140_pneumoni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 scale=0.001 0.001 0.001
- added link left_gripper_link_7; collision box size=0.025 0.03 0.011; visual mesh filename=package://abb_irb140_description/meshes/abb_irb140_pneumoni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 scale=0.001 0.001 0.001
- added link right_gripper_link_1; collision box size=0.025 0.03 0.022; visual mesh filename=package://abb_irb140_description/meshes/abb_irb140_pneumoni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 scale=0.001 0.001 0.001
- added link right_gripper_link_2; collision box size=0.025 0.03 0.011; visual mesh filename=package://abb_irb140_description/meshes/abb_irb140_pneumoni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 scale=0.001 0.001 0.001
- added link right_gripper_link_3; collision box size=0.025 0.03 0.011; visual mesh filename=package://abb_irb140_description/meshes/abb_irb140_pneumoni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 scale=0.001 0.001 0.001
- added link right_gripper_link_4; collision box size=0.025 0.03 0.011; visual mesh filename=package://abb_irb140_description/meshes/abb_irb140_pneumoni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 scale=0.001 0.001 0.001
- added link right_gripper_link_5; collision box size=0.025 0.03 0.011; visual mesh filename=package://abb_irb140_description/meshes/abb_irb140_pneumoni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 scale=0.001 0.001 0.001
- added link right_gripper_link_6; collision box size=0.025 0.03 0.011; visual mesh filename=package://abb_irb140_description/meshes/abb_irb140_pneumoni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 scale=0.001 0.001 0.001
- added link right_gripper_link_7; collision box size=0.025 0.03 0.011; visual mesh filename=package://abb_irb140_description/meshes/abb_irb140_pneumoni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 scale=0.001 0.001 0.001
- link base_link: mass None -> 1.0
Joints:
- added joint left_gripper_base_to_link_1: type fixed, parent base_link, child left_gripper_link_1, origin xyz=0 0 0 rpy=0 0 0
- added joint left_gripper_link_1_to_link_2: type revolute, parent left_gripper_link_1, child left_gripper_link_2, origin xyz=0 0 0 rpy=0 0 0, axis 0 1 0, limit lower=-0.0698 upper=0 effort=10 velocity=1.0
- added joint left_gripper_link_2_to_link_3: type revolute, parent left_gripper_link_2, child left_gripper_link_3, origin xyz=0 0 0 rpy=0 0 0, axis 0 1 0, limit lower=-0.0698 upper=0 effort=10 velocity=1.0
- added joint left_gripper_link_3_to_link_4: type revolute, parent left_gripper_link_3, child left_gripper_link_4, origin xyz=0 0 0 rpy=0 0 0, axis 0 1 0, limit lower=-0.0698 upper=0 effort=10 velocity=1.0
- added joint left_gripper_link_4_to_link_5: type revolute, parent left_gripper_link_4, child left_gripper_link_5, origin xyz=0 0 0 rpy=0 0 0, axis 0 1 0, limit lower=-0.0698 upper=0 effort=10 velocity=1.0
- added joint left_gripper_link_5_to_link_6: type revolute, parent left_gripper_link_5, child left_gripper_link_6, origin xyz=0 0 0 rpy=0 0 0, axis 0 1 0, limit lower=-0.0698 upper=0 effort=10 velocity=1.0
- added joint left_gripper_link_6_to_link_7: type revolute, parent left_gripper_link_6, child left_gripper_link_7, origin xyz=0 0 0 rpy=0 0 0, axis 0 1 0, limit lower=-0.0698 upper=0 effort=10 velocity=1.0
- added joint left_gripper_to_base_link: type fixed, parent base_link, child left_gripper_link_1, origin xyz=0.0 0.046 0.0071 rpy=0.0 0.0 1.57
- added joint right_gripper_base_to_link_1: type fixed, parent base_link, child right_gripper_link_1, origin xyz=0 0 0 rpy=0 0 0
- added joint right_gripper_link_1_to_link_2: type revolute, parent right_gripper_link_1, child right_gripper_link_2, origin xyz=0 0 0 rpy=0 0 0, axis 0 1 0, limit lower=-0.0698 upper=0 effort=10 velocity=1.0
- added joint right_gripper_link_2_to_link_3: type revolute, parent right_gripper_link_2, child right_gripper_link_3, origin xyz=0 0 0 rpy=0 0 0, axis 0 1 0, limit lower=-0.0698 upper=0 effort=10 velocity=1.0
- added joint right_gripper_link_3_to_link_4: type revolute, parent right_gripper_link_3, child right_gripper_link_4, origin xyz=0 0 0 rpy=0 0 0, axis 0 1 0, limit lower=-0.0698 upper=0 effort=10 velocity=1.0
- added joint right_gripper_link_4_to_link_5: type revolute, parent right_gripper_link_4, child right_gripper_link_5, origin xyz=0 0 0 rpy=0 0 0, axis 0 1 0, limit lower=-0.0698 upper=0 effort=10 velocity=1.0
- added joint right_gripper_link_5_to_link_6: type revolute, parent right_gripper_link_5, child right_gripper_link_6, origin xyz=0 0 0 rpy=0 0 0, axis 0 1 0, limit lower=-0.0698 upper=0 effort=10 velocity=1.0
- added joint right_gripper_link_6_to_link_7: type revolute, parent right_gripper_link_6, child right_gripper_link_7, origin xyz=0 0 0 rpy=0 0 0, axis 0 1 0, limit lower=-0.0698 upper=0 effort=10 velocity=1.0
- added joint right_gripper_to_base_link: type fixed, parent base_link, child right_gripper_link_1, origin xyz=-0.008 -0.046 0.0071 rpy=0.0 0.0 -1.57

File: urdf/irb140_pneumonic_gripper_finger.xacro (robot description, xacro)
@@ -1,170 +1,160 @@
 <?xml version="1.0" encoding="UTF-8"?>
 <robot xmlns:xacro="http://www.ros.org/wiki/xacro" name="pneumatic_gripper_finger">
+    <!-- Properties -->
     <xacro:property name="mesh_scale" value="0.001 0.001 0.001"/>
-    <xacro:property mame="collision_scale" value="0.025 0.03 0.1"/>
+    <xacro:property name="collision_scale" value="0.025 0.03 0.1"/>
+    <xacro:property name="joint_lower_limit" value="-0.0698"/>
     <material name="offwhite">
         <color rgba="0.8 0.8 0.8 1"/>
     </material>
-    <!--  Links-->
-    <link name="link_1">
-        <visual>
-            <geometry>
-                <mesh filename="package://abb_irb140_description/meshes/abb_irb140_pneumonic_end_effector/visual/finger_visual/visual/link_1.stl" scale="${mesh_scale}"/>
-            </geometry>
-            <material name="offwhite"/>
-        </visual>
-        <collision>
-            <origin xyz="0 0.005 0.009" rpy=""/>
-            <geometry>
-                <box size="0.025 0.03 0.022"/>
-            </geometry>
-        </collision>
-    </link>
-    <link name="link_1">
-        <visual>
-            <geometry>
-                <mesh filename="package://abb_irb140_description/meshes/abb_irb140_pneumonic_end_effector/visual/finger_visual/visual/link_1.stl" scale="${mesh_scale}"/>
-            </geometry>
-            <material name="offwhite"/>
-        </visual>
-        <collision>
-            <origin xyz="0 0 0.025" rpy="0 0 0"/>
-            <geometry>
-                <box size="0.025 0.03 0.011"/>
-            </geometry>
-        </collision>
-    </link>
-    <link name="link_2">
-        <visual>
-            <geometry>
-                <mesh filename="package://abb_irb140_description/meshes/abb_irb140_pneumonic_end_effector/visual/finger_visual/visual/link_2.stl" scale="${mesh_scale}"/>
-            </geometry>
-            <material name="offwhite"/>
-        </visual>
-        <collision>
-            <origin xyz="0 0 0.035" rpy="0 0 0"/>
-            <geometry>
-                <box size="0.025 0.03 0.011"/>
-            </geometry>
-        </collision>
-    </link>
-    <link name="link_3">
-        <visual>
-            <geometry>
-                <mesh filename="package://abb_irb140_description/meshes/abb_irb140_pneumonic_end_effector/visual/finger_visual/visual/link_3.stl" scale="${mesh_scale}"/>
-            </geometry>
-            <material name="offwhite"/>
-        </visual>
-        <collision>
-            <origin xyz="0 0 0.045" rpy="0 0 0"/>
-            <geometry>
-                <box size="0.025 0.03 0.011"/>
-            </geometry>
-        </collision>
-    </link>
-    <link name="link_4">
-        <visual>
-            <geometry>
-                <mesh filename="package://abb_irb140_description/meshes/abb_irb140_pneumonic_end_effector/visual/finger_visual/visual/link_4.stl" scale="${mesh_scale}"/>
-            </geometry>
-            <material name="offwhite"/>
-        </visual>
-        <collision>
-            <origin xyz="0 0 0.055" rpy="0 0 0"/>
-            <geometry>
-                <box size="0.025 0.03 0.011"/>
-            </geometry>
-        </collision>
-    </link>
-    <link name="link_5">
-        <visual>
-            <geometry>
-                <mesh filename="package://abb_irb140_description/meshes/abb_irb140_pneumonic_end_effector/visual/finger_visual/visual/link_5.stl" scale="${mesh_scale}"/>
-            </geometry>
-            <material name="offwhite"/>
-        </visual>
-        <collision>
-            <origin xyz="0 0 0.065" rpy="0 0 0"/>
-            <geometry>
-                <box size="0.025 0.03 0.011"/>
-            </geometry>
-        </collision>
-    </link>
-    <link name="link_6">
-        <visual>
-            <geometry>
-                <mesh filename="package://abb_irb140_description/meshes/abb_irb140_pneumonic_end_effector/visual/finger_visual/visual/link_6.stl" scale="${mesh_scale}"/>
-            </geometry>
-            <material name="offwhite"/>
-        </visual>
-        <collision>
-            <origin xyz="0 0 0.075" rpy="0 0 0"/>
-            <geometry>
-                <box size="0.025 0.03 0.011"/>
-            </geometry>
-        </collision>
-    </link>
-    <link name="link_7">
-        <visual>
-            <geometry>
-                <mesh filename="package://abb_irb140_description/meshes/abb_irb140_pneumonic_end_effector/visual/finger_visual/visual/link_7.stl" scale="${mesh_scale}"/>
-            </geometry>
-            <material name="offwhite"/>
-        </visual>
-        <collision>
-            <origin xyz="0 0 0.085" rpy="0 0 0"/>
-            <geometry>
-                <box size="0.025 0.03 0.011"/>
-            </geometry>
-        </collision>
-    </link>
-    <!-- Joints -->
-    <joint name="link_1_to_link_2" type="revolute">
-        <parent link="link_1"/>
-        <child link="link_2"/>
-        <!-- joint origin -->
-        <origin xyz="0 0 0/" rpy="0 0 0"/>
-        <axis xyz="0 1 0"/>
-        <limit lower="-0.0524" upper="0" effort="10" velocity="1.0"/>
-    </joint>
-    <joint name="link_2_to_link_3" type="revolute">
-        <parent link="link_2"/>
-        <child link="link_3"/>
-        <!-- joint origin -->
-        <origin xyz="0 0 0/" rpy="0 0 0"/>
-        <axis xyz="0 1 0"/>
-        <limit lower="-0.0524" upper="0" effort="10" velocity="1.0"/>
-    </joint>
-    <joint name="link_3_to_link_4" type="revolute">
-        <parent link="link_3"/>
-        <child link="link_4"/>
-        <!-- joint origin -->
-        <origin xyz="0 0 0/" rpy="0 0 0"/>
-        <axis xyz="0 1 0"/>
-        <limit lower="-0.0524" upper="0" effort="10" velocity="1.0"/>
-    </joint>
-    <joint name="link_4_to_link_5" type="revolute">
-        <parent link="link_4"/>
-        <child link="link_5"/>
-        <!-- joint origin -->
-        <origin xyz="0 0 0/" rpy="0 0 0"/>
-        <axis xyz="0 1 0"/>
-        <limit lower="-0.0524" upper="0" effort="10" velocity="1.0"/>
-    </joint>
-    <joint name="link_5_to_link_6" type="revolute">
-        <parent link="link_5"/>
-        <child link="link_6"/>
-        <!-- joint origin -->
-        <origin xyz="0 0 0/" rpy="0 0 0"/>
-        <axis xyz="0 1 0"/>
-        <limit lower="-0.0524" upper="0" effort="10" velocity="1.0"/>
-    </joint>
-    <joint name="link_6_to_link_7" type="revolute">
-        <parent link="link_6"/>
-        <child link="link_7"/>
-        <!-- joint origin -->
-        <origin xyz="0 0 0/" rpy="0 0 0"/>
-        <axis xyz="0 1 0"/>
-        <limit lower="-0.0524" upper="0" effort="10" velocity="1.0"/>
-    </joint>
+    <!-- Macro for the finger assembly -->
+    <xacro:macro name="pneumatic_gripper_finger" params="name parent">
+        <link name="${name}_link_1">
+            <visual>
+                <geometry>
+                    <mesh filename="package://abb_irb140_description/meshes/abb_irb140_pneumonic_end_effector/visual/finger_visual/visual/link_1.stl" scale="${mesh_scale}"/>
+                </geometry>
+                <material name="offwhite"/>
+            </visual>
+            <collision>
+                <origin xyz="0 0.005 0.009" rpy="0 0 0"/>
+                <geometry>
+                    <box size="0.025 0.03 0.022"/>
+                </geometry>
+            </collision>
+        </link>
+        <link name="${name}_link_2">
+            <visual>
+                <geometry>
+                    <mesh filename="package://abb_irb140_description/meshes/abb_irb140_pneumonic_end_effector/visual/finger_visual/visual/link_2.stl" scale="${mesh_scale}"/>
+                </geometry>
+                <material name="offwhite"/>
+            </visual>
+            <collision>
+                <origin xyz="0 0 0.025" rpy="0 0 0"/>
+                <geometry>
+                    <box size="0.025 0.03 0.011"/>
+                </geometry>
+            </collision>
+        </link>
+        <link name="${name}_link_3">
+            <visual>
+                <geometry>
+                    <mesh filename="package://abb_irb140_description/meshes/abb_irb140_pneumonic_end_effector/visual/finger_visual/visual/link_3.stl" scale="${mesh_scale}"/>
+                </geometry>
+                <material name="offwhite"/>
+            </visual>
+            <collision>
+                <origin xyz="0 0 0.035" rpy="0 0 0"/>
+                <geometry>
+                    <box size="0.025 0.03 0.011"/>
+                </geometry>
+            </collision>
+        </link>
+        <link name="${name}_link_4">
+            <visual>
+                <geometry>
+                    <mesh filename="package://abb_irb140_description/meshes/abb_irb140_pneumonic_end_effector/visual/finger_visual/visual/link_4.stl" scale="${mesh_scale}"/>
+                </geometry>
+                <material name="offwhite"/>
+            </visual>
+            <collision>
+                <origin xyz="0 0 0.055" rpy="0 0 0"/>
+                <geometry>
+                    <box size="0.025 0.03 0.011"/>
+                </geometry>
+            </collision>
+        </link>
+        <link name="${name}_link_5">
+            <visual>
+                <geometry>
+                    <mesh filename="package://abb_irb140_description/meshes/abb_irb140_pneumonic_end_effector/visual/finger_visual/visual/link_5.stl" scale="${mesh_scale}"/>
+                </geometry>
+                <material name="offwhite"/>
+            </visual>
+            <collision>
+                <origin xyz="0 0 0.065" rpy="0 0 0"/>
+                <geometry>
+                    <box size="0.025 0.03 0.011"/>
+                </geometry>
+            </collision>
+        </link>
+        <link name="${name}_link_6">
+            <visual>
+                <geometry>
+                    <mesh filename="package://abb_irb140_description/meshes/abb_irb140_pneumonic_end_effector/visual/finger_visual/visual/link_6.stl" scale="${mesh_scale}"/>
+                </geometry>
+                <material name="offwhite"/>
+            </visual>
+            <collision>
+                <origin xyz="0 0 0.075" rpy="0 0 0"/>
+                <geometry>
+                    <box size="0.025 0.03 0.011"/>
+                </geometry>
+            </collision>
+        </link>
+        <link name="${name}_link_7">
+            <visual>
+                <geometry>
+                    <mesh filename="package://abb_irb140_description/meshes/abb_irb140_pneumonic_end_effector/visual/finger_visual/visual/link_7.stl" scale="${mesh_scale}"/>
+                </geometry>
+                <material name="offwhite"/>
+            </visual>
+            <collision>
+                <origin xyz="0 0 0.085" rpy="0 0 0"/>
+                <geometry>
+                    <box size="0.025 0.03 0.011"/>
+                </geometry>
+            </collision>
+        </link>
+        <!-- Base to link_1 joint -->
+        <joint name="${name}_base_to_link_1" type="fixed">
+            <parent link="${parent}"/>
+            <child link="${name}_link_1"/>
+            <origin xyz="0 0 0" rpy="0 0 0"/>
+        </joint>
+        <!-- Joints between links -->
+        <joint name="${name}_link_1_to_link_2" type="revolute">
+            <parent link="${name}_link_1"/>
+            <child link="${name}_link_2"/>
+            <origin xyz="0 0 0" rpy="0 0 0"/>
+            <axis xyz="0 1 0"/>
+            <limit lower="${joint_lower_limit}" upper="0" effort="10" velocity="1.0"/>
+        </joint>
+        <joint name="${name}_link_2_to_link_3" type="revolute">
+            <parent link="${name}_link_2"/>
+            <child link="${name}_link_3"/>
+            <origin xyz="0 0 0" rpy="0 0 0"/>
+            <axis xyz="0 1 0"/>
+            <limit lower="${joint_lower_limit}" upper="0" effort="10" velocity="1.0"/>
+        </joint>
+        <joint name="${name}_link_3_to_link_4" type="revolute">
+            <parent link="${name}_link_3"/>
+            <child link="${name}_link_4"/>
+            <origin xyz="0 0 0" rpy="0 0 0"/>
+            <axis xyz="0 1 0"/>
+            <limit lower="${joint_lower_limit}" upper="0" effort="10" velocity="1.0"/>
+        </joint>
+        <joint name="${name}_link_4_to_link_5" type="revolute">
+            <parent link="${name}_link_4"/>
+            <child link="${name}_link_5"/>
+            <origin xyz="0 0 0" rpy="0 0 0"/>
+            <axis xyz="0 1 0"/>
+            <limit lower="${joint_lower_limit}" upper="0" effort="10" velocity="1.0"/>
+        </joint>
+        <joint name="${name}_link_5_to_link_6" type="revolute">
+            <parent link="${name}_link_5"/>
+            <child link="${name}_link_6"/>
+            <origin xyz="0 0 0" rpy="0 0 0"/>
+            <axis xyz="0 1 0"/>
+            <limit lower="${joint_lower_limit}" upper="0" effort="10" velocity="1.0"/>
+        </joint>
+        <joint name="${name}_link_6_to_link_7" type="revolute">
+            <parent link="${name}_link_6"/>
+            <child link="${name}_link_7"/>
+            <origin xyz="0 0 0" rpy="0 0 0"/>
+            <axis xyz="0 1 0"/>
+            <limit lower="${joint_lower_limit}" upper="0" effort="10" velocity="1.0"/>
+        </joint>
+    </xacro:macro>
 </robot>
