Commit message: updates

File: urdf/irb140.xacro (robot description, xacro)
@@ -2,4 +2,8 @@
 <robot xmlns:xacro="https://www.ros.org/wiki/xacro" name="abb_irb140">
   <xacro:include filename="$(find abb_irb140_description)/urdf/irb140_pneumonic_gripper.xacro"/>
+  <!-- Path to the ros2_control controller config, consumed by the
+       gz_ros2_control plugin's <parameters> tag below. launch/gazebo.launch.py
+       overrides this with the resolved installed config/controllers.yaml. -->
+  <xacro:arg name="controllers_yaml" default="$(find abb_irb140_description)/config/controllers.yaml"/>
   <material name="abb_orange">
     <color rgba="1 0.43 0 1"/>
@@ -336,12 +340,11 @@
   </ros2_control>
   <!-- Brings up a controller_manager inside gz-sim once the entity is spawned.
-       CONTROLLERS_YAML_PATH is a literal token that launch/gazebo.launch.py
-       rewrites to the installed config/controllers.yaml path before the URDF
-       is published (gz_ros2_control does not evaluate $(find pkg) itself when
-       the description is passed through as plain text). -->
+       The controller config path comes from the controllers_yaml xacro arg
+       (see top of file); launch/gazebo.launch.py passes the resolved installed
+       path since gz_ros2_control does not evaluate $(find pkg) itself. -->
   <gazebo>
     <plugin filename="gz_ros2_control-system"
             name="gz_ros2_control::GazeboSimROS2ControlPlugin">
-      <parameters>CONTROLLERS_YAML_PATH</parameters>
+      <parameters>$(arg controllers_yaml)</parameters>
     </plugin>
   </gazebo>

File: urdf/irb140_pneumonic_gripper.urdf (robot description, URDF)
Before this commit: robot abb_irb140, 27 links, 26 joints
Links:
- removed link base
- removed link base_link
- removed link link_1
- removed link link_2
- removed link link_3
- removed link link_4
- removed link link_5
- removed link link_6
- removed link tool0
Joints:
- removed joint base_link-base
- removed joint joint_1
- removed joint joint_2
- removed joint joint_3
- removed joint joint_4
- removed joint joint_5
- removed joint joint_6
- removed joint joint_6-tool0
- removed joint pneumatic_gripper_to_tool0
- removed joint world-base_link
- added joint pneumatic_gripper_to_world: type fixed, parent world, child pneumatic_gripper_base_link, origin xyz=0 0 0 rpy=0 0 0
- joint depth_camera_to_optical: origin xyz=0 0 0 rpy=0.0 0.0 0 -> xyz=0 0 0 rpy=0 1.57 0
- joint pneumatic_gripper_to_depth_camera: origin xyz=-0.025 0.0 0.05 rpy=3.14159265359 -1.57079632679 0 -> xyz=-0.025 0.0 0.3 rpy=3.14159265359 0 0

File: urdf/irb140_pneumonic_gripper.xacro (robot description, xacro)
@@ -77,5 +77,5 @@
             <parent link="${name}_base_link"/>
             <child link="depth_camera"/>
-            <origin xyz="-0.025 0.0 0.3" rpy="3.14159265359 0 0"/>
+            <origin xyz="-0.025 0.0 0.05" rpy="3.14159265359 -1.57079632679 0"/>
         </joint>
         <!-- Keep depth_camera as its own link/frame in the converted SDF
@@ -93,5 +93,5 @@
             <parent link="depth_camera"/>
             <child link="depth_camera_optical"/>
-            <origin xyz="0 0 0" rpy="0 -1.57 0"/>
+            <origin xyz="0 0 0" rpy="0.0 0.0 0"/>
         </joint>
         <!-- reference="depth_camera" binds the gz-sim sensor to that link.

File: urdf/irb140_pneumonic_gripper_finger.xacro (robot description, xacro)
@@ -35,6 +35,16 @@
          follow a single ros2_control command interface. -->
     <xacro:macro name="pneumatic_gripper_finger" params="name parent mimic_master:='' *origin">
-        <!-- Joint that every non-driver segment of this finger mimics. -->
-        <xacro:property name="_master" value="${mimic_master if mimic_master else name + '_link_1_to_link_2'}"/>
+        <!-- Joint that every non-driver segment of this finger mimics.
+             mimic_master is empty on the driver finger, so it defaults to
+             mimicking its own ${name}_link_1_to_link_2 joint; the other
+             finger passes in the driver's joint name to override that.
+             Written with xacro:unless (rather than a python
+             "X if Y else Z" property expression) so this still parses under
+             JS-based xacro tools (e.g. IDE xacro/URDF previews), not just
+             the Python xacro used at colcon-build time. -->
+        <xacro:property name="_master" value="${name}_link_1_to_link_2"/>
+        <xacro:unless value="${mimic_master == ''}">
+            <xacro:property name="_master" value="${mimic_master}"/>
+        </xacro:unless>
         <link name="${name}_link_1">
             <visual>

Commit message: updates

File: urdf/irb140.xacro (robot description, xacro)
@@ -226,4 +226,9 @@
       <plugin>gz_ros2_control/GazeboSimSystem</plugin>
     </hardware>
+    <!-- initial_value on the position state interface: gz_ros2_control's
+         GazeboSimSystem seeds each joint here when the controller_manager
+         configures (before any controller runs), so the arm spawns in this
+         ready pose instead of the all-zero pose. arm_controller then holds
+         it on activation. All six values are inside the <limit> bounds above. -->
     <joint name="joint_1">
       <command_interface name="position">
@@ -231,5 +236,7 @@
         <param name="max">3.1416</param>
       </command_interface>
-      <state_interface name="position"/>
+      <state_interface name="position">
+        <param name="initial_value">0.0</param>
+      </state_interface>
       <state_interface name="velocity"/>
     </joint>
@@ -239,5 +246,7 @@
         <param name="max">1.9199</param>
       </command_interface>
-      <state_interface name="position"/>
+      <state_interface name="position">
+        <param name="initial_value">0.0873</param>
+      </state_interface>
       <state_interface name="velocity"/>
     </joint>
@@ -247,5 +256,7 @@
         <param name="max">1.1345</param>
       </command_interface>
-      <state_interface name="position"/>
+      <state_interface name="position">
+        <param name="initial_value">-0.283605</param>
+      </state_interface>
       <state_interface name="velocity"/>
     </joint>
@@ -255,5 +266,7 @@
         <param name="max">3.49</param>
       </command_interface>
-      <state_interface name="position"/>
+      <state_interface name="position">
+        <param name="initial_value">0.0</param>
+      </state_interface>
       <state_interface name="velocity"/>
     </joint>
@@ -263,5 +276,7 @@
         <param name="max">2.0944</param>
       </command_interface>
-      <state_interface name="position"/>
+      <state_interface name="position">
+        <param name="initial_value">1.256640</param>
+      </state_interface>
       <state_interface name="velocity"/>
     </joint>
@@ -271,5 +286,7 @@
         <param name="max">6.9813</param>
       </command_interface>
-      <state_interface name="position"/>
+      <state_interface name="position">
+        <param name="initial_value">0.0</param>
+      </state_interface>
       <state_interface name="velocity"/>
     </joint>
