Commit message: updated scale of abb irb robot to be in proportion with actual measurements

File: urdf/irb140.urdf (robot description, URDF)
Before this commit: robot abb_irb140, 10 links, 9 joints
Links:
- link base_link: geometry collision mesh filename=package://abb_irb140_description/meshes/abb_irb140/collisio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 scale=0.208333 0.208333 0.208333; visual mesh filename=package://abb_irb140_description/meshes/abb_irb140/visual/b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 scale=0.208333 0.208333 0.208333
- link link_1: geometry collision mesh filename=package://abb_irb140_description/meshes/abb_irb140/collisio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 scale=0.208333 0.208333 0.208333; visual mesh filename=package://abb_irb140_description/meshes/abb_irb140/visual/l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 scale=0.208333 0.208333 0.208333
- link link_2: geometry collision mesh filename=package://abb_irb140_description/meshes/abb_irb140/collisio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 scale=0.208333 0.208333 0.208333; visual mesh filename=package://abb_irb140_description/meshes/abb_irb140/visual/l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 scale=0.208333 0.208333 0.208333
- link link_3: geometry collision mesh filename=package://abb_irb140_description/meshes/abb_irb140/collisio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 scale=0.208333 0.208333 0.208333; visual mesh filename=package://abb_irb140_description/meshes/abb_irb140/visual/l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 scale=0.208333 0.208333 0.208333
- link link_4: geometry collision mesh filename=package://abb_irb140_description/meshes/abb_irb140/collisio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 scale=0.208333 0.208333 0.208333; visual mesh filename=package://abb_irb140_description/meshes/abb_irb140/visual/l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 scale=0.208333 0.208333 0.208333
- link link_5: geometry collision mesh filename=package://abb_irb140_description/meshes/abb_irb140/collisio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 scale=0.208333 0.208333 0.208333; visual mesh filename=package://abb_irb140_description/meshes/abb_irb140/visual/l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 scale=0.208333 0.208333 0.208333
- link link_6: geometry collision mesh filename=package://abb_irb140_description/meshes/abb_irb140/collisio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 scale=0.208333 0.208333 0.208333; visual mesh filename=package://abb_irb140_description/meshes/abb_irb140/visual/l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 scale=0.208333 0.208333 0.208333
Joints:
- joint joint_2: origin xyz=0.28 0 1.38 rpy=0 0 0 -> xyz=0.058333 0 0.2875 rpy=0 0 0
- joint joint_3: origin xyz=0 0 1.42 rpy=0 0 0 -> xyz=0 0 0.295833 rpy=0 0 0
- joint joint_5: origin xyz=1.49 0 0 rpy=0 0 0 -> xyz=0.310417 0 0 rpy=0 0 0
- joint joint_6: origin xyz=0 0 0.02 rpy=0 0 0 -> xyz=0 0 0.004167 rpy=0 0 0

Commit message: added depth camera links and joints for the standard abb robot configuration

File: urdf/irb140.urdf (robot description, URDF)
Before this commit: robot abb_irb140, 10 links, 9 joints
Links:
- added link depth_camera
- added link depth_camera_optical
Joints:
- added joint depth_camera-optical: type fixed, parent tool0, child depth_camera_optical, origin xyz=0 0 0.05 rpy=0 -1.5707963268 0
- added joint tool0-depth_camera: type fixed, parent tool0, child depth_camera, origin xyz=0.0 0 0.05 rpy=0 -1.57079632679 0

Commit message: updates

File: urdf/irb140.urdf (robot description, URDF)
Before this commit: robot abb_irb140, 12 links, 11 joints
Links:
- removed link depth_camera
- removed link depth_camera_optical
- added link pneumatic_gripper_1_base_link, mass 1.0; collision box size=0.1 0.125 0.062; visual mesh filename=package://abb_irb140_description/meshes/abb_irb140_pneumoni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 scale=0.001 0.001 0.001
- added link pneumatic_gripper_1_left_link_1; collision box size=0.025 0.03 0.022; visual mesh filename=package://abb_irb140_description/meshes/abb_irb140_pneumoni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 scale=0.001 0.001 0.001
- added link pneumatic_gripper_1_left_link_2; collision box size=0.025 0.03 0.011; visual mesh filename=package://abb_irb140_description/meshes/abb_irb140_pneumoni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 scale=0.001 0.001 0.001
- added link pneumatic_gripper_1_left_link_3; collision box size=0.025 0.03 0.011; visual mesh filename=package://abb_irb140_description/meshes/abb_irb140_pneumoni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 scale=0.001 0.001 0.001
- added link pneumatic_gripper_1_left_link_4; collision box size=0.025 0.03 0.011; visual mesh filename=package://abb_irb140_description/meshes/abb_irb140_pneumoni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 scale=0.001 0.001 0.001
- added link pneumatic_gripper_1_left_link_5; collision box size=0.025 0.03 0.011; visual mesh filename=package://abb_irb140_description/meshes/abb_irb140_pneumoni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 scale=0.001 0.001 0.001
- added link pneumatic_gripper_1_left_link_6; collision box size=0.025 0.03 0.011; visual mesh filename=package://abb_irb140_description/meshes/abb_irb140_pneumoni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 scale=0.001 0.001 0.001
- added link pneumatic_gripper_1_left_link_7; collision box size=0.025 0.03 0.011; visual mesh filename=package://abb_irb140_description/meshes/abb_irb140_pneumoni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 scale=0.001 0.001 0.001
- added link pneumatic_gripper_1_right_link_1; collision box size=0.025 0.03 0.022; visual mesh filename=package://abb_irb140_description/meshes/abb_irb140_pneumoni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 scale=0.001 0.001 0.001
- added link pneumatic_gripper_1_right_link_2; collision box size=0.025 0.03 0.011; visual mesh filename=package://abb_irb140_description/meshes/abb_irb140_pneumoni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 scale=0.001 0.001 0.001
- added link pneumatic_gripper_1_right_link_3; collision box size=0.025 0.03 0.011; visual mesh filename=package://abb_irb140_description/meshes/abb_irb140_pneumoni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 scale=0.001 0.001 0.001
- added link pneumatic_gripper_1_right_link_4; collision box size=0.025 0.03 0.011; visual mesh filename=package://abb_irb140_description/meshes/abb_irb140_pneumoni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 scale=0.001 0.001 0.001
- added link pneumatic_gripper_1_right_link_5; collision box size=0.025 0.03 0.011; visual mesh filename=package://abb_irb140_description/meshes/abb_irb140_pneumoni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 scale=0.001 0.001 0.001
- added link pneumatic_gripper_1_right_link_6; collision box size=0.025 0.03 0.011; visual mesh filename=package://abb_irb140_description/meshes/abb_irb140_pneumoni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 scale=0.001 0.001 0.001
- added link pneumatic_gripper_1_right_link_7; collision box size=0.025 0.03 0.011; visual mesh filename=package://abb_irb140_description/meshes/abb_irb140_pneumoni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 scale=0.001 0.001 0.001
Joints:
- removed joint depth_camera-optical
- removed joint tool0-depth_camera
- added joint pneumatic_gripper_1_left_base_to_link_1: type fixed, parent pneumatic_gripper_1_base_link, child pneumatic_gripper_1_left_link_1, origin xyz=0.0 0.046 0.0071 rpy=0.0 0.0 1.57
- added joint pneumatic_gripper_1_left_link_1_to_link_2: type revolute, parent pneumatic_gripper_1_left_link_1, child pneumatic_gripper_1_left_link_2, origin xyz=0 0 0 rpy=0 0 0, axis 0 1 0, limit lower=-0.0698 upper=0 effort=10 velocity=1.0
- added joint pneumatic_gripper_1_left_link_2_to_link_3: type revolute, parent pneumatic_gripper_1_left_link_2, child pneumatic_gripper_1_left_link_3, origin xyz=0 0 0 rpy=0 0 0, axis 0 1 0, limit lower=-0.0698 upper=0 effort=10 velocity=1.0
- added joint pneumatic_gripper_1_left_link_3_to_link_4: type revolute, parent pneumatic_gripper_1_left_link_3, child pneumatic_gripper_1_left_link_4, origin xyz=0 0 0 rpy=0 0 0, axis 0 1 0, limit lower=-0.0698 upper=0 effort=10 velocity=1.0
- added joint pneumatic_gripper_1_left_link_4_to_link_5: type revolute, parent pneumatic_gripper_1_left_link_4, child pneumatic_gripper_1_left_link_5, origin xyz=0 0 0 rpy=0 0 0, axis 0 1 0, limit lower=-0.0698 upper=0 effort=10 velocity=1.0
- added joint pneumatic_gripper_1_left_link_5_to_link_6: type revolute, parent pneumatic_gripper_1_left_link_5, child pneumatic_gripper_1_left_link_6, origin xyz=0 0 0 rpy=0 0 0, axis 0 1 0, limit lower=-0.0698 upper=0 effort=10 velocity=1.0
- added joint pneumatic_gripper_1_left_link_6_to_link_7: type revolute, parent pneumatic_gripper_1_left_link_6, child pneumatic_gripper_1_left_link_7, origin xyz=0 0 0 rpy=0 0 0, axis 0 1 0, limit lower=-0.0698 upper=0 effort=10 velocity=1.0
- added joint pneumatic_gripper_1_right_base_to_link_1: type fixed, parent pneumatic_gripper_1_base_link, child pneumatic_gripper_1_right_link_1, origin xyz=-0.008 -0.046 0.0071 rpy=0.0 0.0 -1.57
- added joint pneumatic_gripper_1_right_link_1_to_link_2: type revolute, parent pneumatic_gripper_1_right_link_1, child pneumatic_gripper_1_right_link_2, origin xyz=0 0 0 rpy=0 0 0, axis 0 1 0, limit lower=-0.0698 upper=0 effort=10 velocity=1.0
- added joint pneumatic_gripper_1_right_link_2_to_link_3: type revolute, parent pneumatic_gripper_1_right_link_2, child pneumatic_gripper_1_right_link_3, origin xyz=0 0 0 rpy=0 0 0, axis 0 1 0, limit lower=-0.0698 upper=0 effort=10 velocity=1.0
- added joint pneumatic_gripper_1_right_link_3_to_link_4: type revolute, parent pneumatic_gripper_1_right_link_3, child pneumatic_gripper_1_right_link_4, origin xyz=0 0 0 rpy=0 0 0, axis 0 1 0, limit lower=-0.0698 upper=0 effort=10 velocity=1.0
- added joint pneumatic_gripper_1_right_link_4_to_link_5: type revolute, parent pneumatic_gripper_1_right_link_4, child pneumatic_gripper_1_right_link_5, origin xyz=0 0 0 rpy=0 0 0, axis 0 1 0, limit lower=-0.0698 upper=0 effort=10 velocity=1.0
- added joint pneumatic_gripper_1_right_link_5_to_link_6: type revolute, parent pneumatic_gripper_1_right_link_5, child pneumatic_gripper_1_right_link_6, origin xyz=0 0 0 rpy=0 0 0, axis 0 1 0, limit lower=-0.0698 upper=0 effort=10 velocity=1.0
- added joint pneumatic_gripper_1_right_link_6_to_link_7: type revolute, parent pneumatic_gripper_1_right_link_6, child pneumatic_gripper_1_right_link_7, origin xyz=0 0 0 rpy=0 0 0, axis 0 1 0, limit lower=-0.0698 upper=0 effort=10 velocity=1.0
- added joint pneumatic_gripper_1_to_tool0: type fixed, parent tool0, child pneumatic_gripper_1_base_link, origin xyz=0 0 0 rpy=0 0 0

File: urdf/irb140_pneumonic_gripper.xacro (robot description, xacro)
@@ -2,37 +2,41 @@
 <robot xmlns:xacro="http://www.ros.org/wiki/xacro" name="pneumatic_gripper">
 <xacro:include filename="$(find abb_irb140_description)/urdf/irb140_pneumonic_gripper_finger.xacro"/>
-<link name="base_link">
-    <visual>
-        <origin xyz="0 0 -0.03105" rpy="0 0 0"/>
-        <geometry>
-            <mesh filename="package://abb_irb140_description/meshes/abb_irb140_pneumonic_end_effector/visual/ABBIRB140_EndEffector.stl" scale="0.001 0.001 0.001"/>
-        </geometry>
-        <material name="plastic">
-            <color rgba="0.11 0.11 0.11 1"/>
-        </material>
-    </visual>
-    <collision>
-        <origin xyz="0.0165 0 -0.005" rpy="0 0 0"/>
-        <geometry>
-            <box size="0.1 0.125 0.062"/>
-        </geometry>
-    </collision>
-    <inertial>
-        <mass value="1.0"/>
-        <inertia ixx="0.001" ixy="0" ixz="0" iyy="0.001" iyz="0" izz="0.001"/>
-    </inertial>
-</link>
-<!-- Spawn left and right gripper fingers -->
-<xacro:pneumatic_gripper_finger name="left_gripper" parent="base_link"/>
-<xacro:pneumatic_gripper_finger name="right_gripper" parent="base_link"/>
-<joint name="left_gripper_to_base_link" type="fixed">
-    <parent link="base_link"/>
-    <child link="left_gripper_link_1"/>
-    <origin xyz="0.0 0.046 0.0071" rpy="0.0 0.0 1.57"/>
-</joint>
-<joint name="right_gripper_to_base_link" type="fixed">
-    <parent link="base_link"/>
-    <child link="right_gripper_link_1"/>
-    <origin xyz="-0.008 -0.046 0.0071" rpy="0.0 0.0 -1.57"/>
-</joint>
+<xacro:macro name="pneumatic_gripper" params="name parent">
+    <!-- Attach the gripper body to the robot flange -->
+    <joint name="${name}_to_${parent}" type="fixed">
+        <parent link="${parent}"/>
+        <child link="${name}_base_link"/>
+        <origin xyz="0 0 0" rpy="0 0 0"/>
+    </joint>
+    <link name="${name}_base_link">
+        <visual>
+            <origin xyz="0 0 -0.03105" rpy="0 0 0"/>
+            <geometry>
+                <mesh filename="package://abb_irb140_description/meshes/abb_irb140_pneumonic_end_effector/visual/ABBIRB140_EndEffector.stl" scale="0.001 0.001 0.001"/>
+            </geometry>
+            <material name="plastic">
+                <color rgba="0.11 0.11 0.11 1"/>
+            </material>
+        </visual>
+        <collision>
+            <origin xyz="0.0165 0 -0.005" rpy="0 0 0"/>
+            <geometry>
+                <box size="0.1 0.125 0.062"/>
+            </geometry>
+        </collision>
+        <inertial>
+            <mass value="1.0"/>
+            <inertia ixx="0.001" ixy="0" ixz="0" iyy="0.001" iyz="0" izz="0.001"/>
+        </inertial>
+    </link>
+    <!-- Spawn left and right gripper fingers.
+         The offset/rotation for each finger is passed straight into the
+         finger macro's base joint (its <origin> block). -->
+    <xacro:pneumatic_gripper_finger name="${name}_left" parent="${name}_base_link">
+        <origin xyz="0.0 0.046 0.0071" rpy="0.0 0.0 1.57"/>
+    </xacro:pneumatic_gripper_finger>
+    <xacro:pneumatic_gripper_finger name="${name}_right" parent="${name}_base_link">
+        <origin xyz="-0.008 -0.046 0.0071" rpy="0.0 0.0 -1.57"/>
+    </xacro:pneumatic_gripper_finger>
+</xacro:macro>
 </robot>

File: urdf/irb140_pneumonic_gripper_finger.xacro (robot description, xacro)
@@ -9,5 +9,5 @@
     </material>
     <!-- Macro for the finger assembly -->
-    <xacro:macro name="pneumatic_gripper_finger" params="name parent">
+    <xacro:macro name="pneumatic_gripper_finger" params="name parent *origin">
         <link name="${name}_link_1">
             <visual>
@@ -112,5 +112,5 @@
             <parent link="${parent}"/>
             <child link="${name}_link_1"/>
-            <origin xyz="0 0 0" rpy="0 0 0"/>
+            <xacro:insert_block name="origin"/>
         </joint>
         <!-- Joints between links -->

Commit message: updates

File: urdf/irb140.urdf (robot description, URDF)
Before this commit: robot abb_irb140, 25 links, 24 joints
Links:
- removed link pneumatic_gripper_1_base_link
- removed link pneumatic_gripper_1_left_link_1
- removed link pneumatic_gripper_1_left_link_2
- removed link pneumatic_gripper_1_left_link_3
- removed link pneumatic_gripper_1_left_link_4
- removed link pneumatic_gripper_1_left_link_5
- removed link pneumatic_gripper_1_left_link_6
- removed link pneumatic_gripper_1_left_link_7
- removed link pneumatic_gripper_1_right_link_1
- removed link pneumatic_gripper_1_right_link_2
- removed link pneumatic_gripper_1_right_link_3
- removed link pneumatic_gripper_1_right_link_4
- removed link pneumatic_gripper_1_right_link_5
- removed link pneumatic_gripper_1_right_link_6
- removed link pneumatic_gripper_1_right_link_7
- added link pneumatic_gripper_base_link, mass 1.0; collision box size=0.1 0.125 0.062; visual mesh filename=package://abb_irb140_description/meshes/abb_irb140_pneumoni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 scale=0.001 0.001 0.001
- added link pneumatic_gripper_left_link_1; collision box size=0.025 0.03 0.022; visual mesh filename=package://abb_irb140_description/meshes/abb_irb140_pneumoni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 scale=0.001 0.001 0.001
- added link pneumatic_gripper_left_link_2; collision box size=0.025 0.03 0.011; visual mesh filename=package://abb_irb140_description/meshes/abb_irb140_pneumoni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 scale=0.001 0.001 0.001
- added link pneumatic_gripper_left_link_3; collision box size=0.025 0.03 0.011; visual mesh filename=package://abb_irb140_description/meshes/abb_irb140_pneumoni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 scale=0.001 0.001 0.001
- added link pneumatic_gripper_left_link_4; collision box size=0.025 0.03 0.011; visual mesh filename=package://abb_irb140_description/meshes/abb_irb140_pneumoni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 scale=0.001 0.001 0.001
- added link pneumatic_gripper_left_link_5; collision box size=0.025 0.03 0.011; visual mesh filename=package://abb_irb140_description/meshes/abb_irb140_pneumoni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 scale=0.001 0.001 0.001
- added link pneumatic_gripper_left_link_6; collision box size=0.025 0.03 0.011; visual mesh filename=package://abb_irb140_description/meshes/abb_irb140_pneumoni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 scale=0.001 0.001 0.001
- added link pneumatic_gripper_left_link_7; collision box size=0.025 0.03 0.011; visual mesh filename=package://abb_irb140_description/meshes/abb_irb140_pneumoni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 scale=0.001 0.001 0.001
- added link pneumatic_gripper_right_link_1; collision box size=0.025 0.03 0.022; visual mesh filename=package://abb_irb140_description/meshes/abb_irb140_pneumoni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 scale=0.001 0.001 0.001
- added link pneumatic_gripper_right_link_2; collision box size=0.025 0.03 0.011; visual mesh filename=package://abb_irb140_description/meshes/abb_irb140_pneumoni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 scale=0.001 0.001 0.001
- added link pneumatic_gripper_right_link_3; collision box size=0.025 0.03 0.011; visual mesh filename=package://abb_irb140_description/meshes/abb_irb140_pneumoni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 scale=0.001 0.001 0.001
- added link pneumatic_gripper_right_link_4; collision box size=0.025 0.03 0.011; visual mesh filename=package://abb_irb140_description/meshes/abb_irb140_pneumoni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 scale=0.001 0.001 0.001
- added link pneumatic_gripper_right_link_5; collision box size=0.025 0.03 0.011; visual mesh filename=package://abb_irb140_description/meshes/abb_irb140_pneumoni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 scale=0.001 0.001 0.001
- added link pneumatic_gripper_right_link_6; collision box size=0.025 0.03 0.011; visual mesh filename=package://abb_irb140_description/meshes/abb_irb140_pneumoni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 scale=0.001 0.001 0.001
- added link pneumatic_gripper_right_link_7; collision box size=0.025 0.03 0.011; visual mesh filename=package://abb_irb140_description/meshes/abb_irb140_pneumoni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 scale=0.001 0.001 0.001
Joints:
- removed joint pneumatic_gripper_1_left_base_to_link_1
- removed joint pneumatic_gripper_1_left_link_1_to_link_2
- removed joint pneumatic_gripper_1_left_link_2_to_link_3
- removed joint pneumatic_gripper_1_left_link_3_to_link_4
- removed joint pneumatic_gripper_1_left_link_4_to_link_5
- removed joint pneumatic_gripper_1_left_link_5_to_link_6
- removed joint pneumatic_gripper_1_left_link_6_to_link_7
- removed joint pneumatic_gripper_1_right_base_to_link_1
- removed joint pneumatic_gripper_1_right_link_1_to_link_2
- removed joint pneumatic_gripper_1_right_link_2_to_link_3
- removed joint pneumatic_gripper_1_right_link_3_to_link_4
- removed joint pneumatic_gripper_1_right_link_4_to_link_5
- removed joint pneumatic_gripper_1_right_link_5_to_link_6
- removed joint pneumatic_gripper_1_right_link_6_to_link_7
- removed joint pneumatic_gripper_1_to_tool0
- added joint pneumatic_gripper_left_base_to_link_1: type fixed, parent pneumatic_gripper_base_link, child pneumatic_gripper_left_link_1, origin xyz=0.0 0.046 0.0071 rpy=0.0 0.0 1.57
- added joint pneumatic_gripper_left_link_1_to_link_2: type revolute, parent pneumatic_gripper_left_link_1, child pneumatic_gripper_left_link_2, origin xyz=0 0 0 rpy=0 0 0, axis 0 1 0, limit lower=-0.0698 upper=0 effort=10 velocity=1.0
- added joint pneumatic_gripper_left_link_2_to_link_3: type revolute, parent pneumatic_gripper_left_link_2, child pneumatic_gripper_left_link_3, origin xyz=0 0 0 rpy=0 0 0, axis 0 1 0, limit lower=-0.0698 upper=0 effort=10 velocity=1.0
- added joint pneumatic_gripper_left_link_3_to_link_4: type revolute, parent pneumatic_gripper_left_link_3, child pneumatic_gripper_left_link_4, origin xyz=0 0 0 rpy=0 0 0, axis 0 1 0, limit lower=-0.0698 upper=0 effort=10 velocity=1.0
- added joint pneumatic_gripper_left_link_4_to_link_5: type revolute, parent pneumatic_gripper_left_link_4, child pneumatic_gripper_left_link_5, origin xyz=0 0 0 rpy=0 0 0, axis 0 1 0, limit lower=-0.0698 upper=0 effort=10 velocity=1.0
- added joint pneumatic_gripper_left_link_5_to_link_6: type revolute, parent pneumatic_gripper_left_link_5, child pneumatic_gripper_left_link_6, origin xyz=0 0 0 rpy=0 0 0, axis 0 1 0, limit lower=-0.0698 upper=0 effort=10 velocity=1.0
- added joint pneumatic_gripper_left_link_6_to_link_7: type revolute, parent pneumatic_gripper_left_link_6, child pneumatic_gripper_left_link_7, origin xyz=0 0 0 rpy=0 0 0, axis 0 1 0, limit lower=-0.0698 upper=0 effort=10 velocity=1.0
- added joint pneumatic_gripper_right_base_to_link_1: type fixed, parent pneumatic_gripper_base_link, child pneumatic_gripper_right_link_1, origin xyz=-0.008 -0.046 0.0071 rpy=0.0 0.0 -1.57
- added joint pneumatic_gripper_right_link_1_to_link_2: type revolute, parent pneumatic_gripper_right_link_1, child pneumatic_gripper_right_link_2, origin xyz=0 0 0 rpy=0 0 0, axis 0 1 0, limit lower=-0.0698 upper=0 effort=10 velocity=1.0
- added joint pneumatic_gripper_right_link_2_to_link_3: type revolute, parent pneumatic_gripper_right_link_2, child pneumatic_gripper_right_link_3, origin xyz=0 0 0 rpy=0 0 0, axis 0 1 0, limit lower=-0.0698 upper=0 effort=10 velocity=1.0
- added joint pneumatic_gripper_right_link_3_to_link_4: type revolute, parent pneumatic_gripper_right_link_3, child pneumatic_gripper_right_link_4, origin xyz=0 0 0 rpy=0 0 0, axis 0 1 0, limit lower=-0.0698 upper=0 effort=10 velocity=1.0
- added joint pneumatic_gripper_right_link_4_to_link_5: type revolute, parent pneumatic_gripper_right_link_4, child pneumatic_gripper_right_link_5, origin xyz=0 0 0 rpy=0 0 0, axis 0 1 0, limit lower=-0.0698 upper=0 effort=10 velocity=1.0
- added joint pneumatic_gripper_right_link_5_to_link_6: type revolute, parent pneumatic_gripper_right_link_5, child pneumatic_gripper_right_link_6, origin xyz=0 0 0 rpy=0 0 0, axis 0 1 0, limit lower=-0.0698 upper=0 effort=10 velocity=1.0
- added joint pneumatic_gripper_right_link_6_to_link_7: type revolute, parent pneumatic_gripper_right_link_6, child pneumatic_gripper_right_link_7, origin xyz=0 0 0 rpy=0 0 0, axis 0 1 0, limit lower=-0.0698 upper=0 effort=10 velocity=1.0
- added joint pneumatic_gripper_to_tool0: type fixed, parent tool0, child pneumatic_gripper_base_link, origin xyz=0.05 0 0 rpy=0 0 0

File: urdf/irb140.xacro (robot description, xacro)
@@ -210,4 +210,4 @@
     <child link="base"/>
   </joint>
-  <xacro:pneumatic_gripper name="pneumatic_gripper_1" parent="tool0"/>
+  <xacro:pneumatic_gripper name="pneumatic_gripper" parent="tool0" xyz="0.00 0.0 0.08" rpy="0 0 3.142"/>
 </robot>

File: urdf/irb140_pneumonic_gripper.xacro (robot description, xacro)
@@ -2,10 +2,12 @@
 <robot xmlns:xacro="http://www.ros.org/wiki/xacro" name="pneumatic_gripper">
 <xacro:include filename="$(find abb_irb140_description)/urdf/irb140_pneumonic_gripper_finger.xacro"/>
-<xacro:macro name="pneumatic_gripper" params="name parent">
-    <!-- Attach the gripper body to the robot flange -->
+<xacro:macro name="pneumatic_gripper" params="name parent xyz:='0 0 0' rpy:='0 0 0'">
+    <!-- Attach the gripper body to the robot flange.
+         xyz/rpy are expressed in the parent (tool0) frame; set xyz to
+         shift the gripper along the flange axes. -->
     <joint name="${name}_to_${parent}" type="fixed">
         <parent link="${parent}"/>
         <child link="${name}_base_link"/>
-        <origin xyz="0 0 0" rpy="0 0 0"/>
+        <origin xyz="${xyz}" rpy="${rpy}"/>
     </joint>
     <link name="${name}_base_link">
@@ -39,4 +41,5 @@
         <origin xyz="-0.008 -0.046 0.0071" rpy="0.0 0.0 -1.57"/>
     </xacro:pneumatic_gripper_finger>
+    <xacro:arg name="include_camera" default="true"/>
 </xacro:macro>
 </robot>

Commit message: updates

File: urdf/irb140.urdf (robot description, URDF)
Before this commit: robot abb_irb140, 25 links, 24 joints
Joints:
- joint pneumatic_gripper_to_tool0: origin xyz=0.05 0 0 rpy=0 0 0 -> xyz=0.00 0.0 0.08 rpy=0 0 3.142
