Commit message: updates

File: urdf/irb140.urdf (robot description, URDF)
Before this commit: robot abb_irb140, 25 links, 24 joints
Links:
- added link depth_camera, mass 0.05
- added link depth_camera_optical
- link pneumatic_gripper_base_link: mass 1.0 -> 0.50375
- link pneumatic_gripper_left_link_1: mass None -> 0.01815
- link pneumatic_gripper_left_link_2: mass None -> 0.009075
- link pneumatic_gripper_left_link_3: mass None -> 0.009075
- link pneumatic_gripper_left_link_4: mass None -> 0.009075
- link pneumatic_gripper_left_link_5: mass None -> 0.009075
- link pneumatic_gripper_left_link_6: mass None -> 0.009075
- link pneumatic_gripper_left_link_7: mass None -> 0.009075
- link pneumatic_gripper_right_link_1: mass None -> 0.01815
- link pneumatic_gripper_right_link_2: mass None -> 0.009075
- link pneumatic_gripper_right_link_3: mass None -> 0.009075
- link pneumatic_gripper_right_link_4: mass None -> 0.009075
- link pneumatic_gripper_right_link_5: mass None -> 0.009075
- link pneumatic_gripper_right_link_6: mass None -> 0.009075
- link pneumatic_gripper_right_link_7: mass None -> 0.009075
Joints:
- added joint depth_camera_to_optical: type fixed, parent depth_camera, child depth_camera_optical, origin xyz=0 0 0 rpy=0 0 0
- added joint pneumatic_gripper_to_depth_camera: type fixed, parent pneumatic_gripper_base_link, child depth_camera, origin xyz=-0.025 0.0 0.3 rpy=3.14159265359 0 0
- joint pneumatic_gripper_left_link_1_to_link_2: limit lower=-0.0698 upper=0 effort=10 velocity=1.0 -> lower=-0.09 upper=0 effort=10 velocity=1.0
- joint pneumatic_gripper_left_link_2_to_link_3: limit lower=-0.0698 upper=0 effort=10 velocity=1.0 -> lower=-0.09 upper=0 effort=10 velocity=1.0; mimic (none) -> joint=pneumatic_gripper_left_link_1_to_link_2 multiplier=1.0 offset=0.0
- joint pneumatic_gripper_left_link_3_to_link_4: limit lower=-0.0698 upper=0 effort=10 velocity=1.0 -> lower=-0.09 upper=0 effort=10 velocity=1.0; mimic (none) -> joint=pneumatic_gripper_left_link_1_to_link_2 multiplier=1.0 offset=0.0
- joint pneumatic_gripper_left_link_4_to_link_5: limit lower=-0.0698 upper=0 effort=10 velocity=1.0 -> lower=-0.09 upper=0 effort=10 velocity=1.0; mimic (none) -> joint=pneumatic_gripper_left_link_1_to_link_2 multiplier=1.0 offset=0.0
- joint pneumatic_gripper_left_link_5_to_link_6: limit lower=-0.0698 upper=0 effort=10 velocity=1.0 -> lower=-0.09 upper=0 effort=10 velocity=1.0; mimic (none) -> joint=pneumatic_gripper_left_link_1_to_link_2 multiplier=1.0 offset=0.0
- joint pneumatic_gripper_left_link_6_to_link_7: limit lower=-0.0698 upper=0 effort=10 velocity=1.0 -> lower=-0.09 upper=0 effort=10 velocity=1.0; mimic (none) -> joint=pneumatic_gripper_left_link_1_to_link_2 multiplier=1.0 offset=0.0
- joint pneumatic_gripper_right_link_1_to_link_2: limit lower=-0.0698 upper=0 effort=10 velocity=1.0 -> lower=-0.09 upper=0 effort=10 velocity=1.0; mimic (none) -> joint=pneumatic_gripper_left_link_1_to_link_2 multiplier=1.0 offset=0.0
- joint pneumatic_gripper_right_link_2_to_link_3: limit lower=-0.0698 upper=0 effort=10 velocity=1.0 -> lower=-0.09 upper=0 effort=10 velocity=1.0; mimic (none) -> joint=pneumatic_gripper_left_link_1_to_link_2 multiplier=1.0 offset=0.0
- joint pneumatic_gripper_right_link_3_to_link_4: limit lower=-0.0698 upper=0 effort=10 velocity=1.0 -> lower=-0.09 upper=0 effort=10 velocity=1.0; mimic (none) -> joint=pneumatic_gripper_left_link_1_to_link_2 multiplier=1.0 offset=0.0
- joint pneumatic_gripper_right_link_4_to_link_5: limit lower=-0.0698 upper=0 effort=10 velocity=1.0 -> lower=-0.09 upper=0 effort=10 velocity=1.0; mimic (none) -> joint=pneumatic_gripper_left_link_1_to_link_2 multiplier=1.0 offset=0.0
- joint pneumatic_gripper_right_link_5_to_link_6: limit lower=-0.0698 upper=0 effort=10 velocity=1.0 -> lower=-0.09 upper=0 effort=10 velocity=1.0; mimic (none) -> joint=pneumatic_gripper_left_link_1_to_link_2 multiplier=1.0 offset=0.0
- joint pneumatic_gripper_right_link_6_to_link_7: limit lower=-0.0698 upper=0 effort=10 velocity=1.0 -> lower=-0.09 upper=0 effort=10 velocity=1.0; mimic (none) -> joint=pneumatic_gripper_left_link_1_to_link_2 multiplier=1.0 offset=0.0

File: urdf/irb140.xacro (robot description, xacro)
@@ -211,3 +211,138 @@
   </joint>
   <xacro:pneumatic_gripper name="pneumatic_gripper" parent="tool0" xyz="0.00 0.0 0.08" rpy="0 0 3.142"/>
+  <!-- =================================================================== -->
+  <!-- ros2_control + Gazebo Sim                                           -->
+  <!-- =================================================================== -->
+  <!-- ros2_control hardware for the 6 arm joints. gz_ros2_control's
+       GazeboSimSystem reads/writes these interfaces straight from the gz-sim
+       physics engine. command/state interfaces match config/controllers.yaml
+       (arm_controller: position command; position + velocity state). -->
+  <ros2_control name="GazeboSimSystem" type="system">
+    <hardware>
+      <plugin>gz_ros2_control/GazeboSimSystem</plugin>
+    </hardware>
+    <joint name="joint_1">
+      <command_interface name="position">
+        <param name="min">-3.1416</param>
+        <param name="max">3.1416</param>
+      </command_interface>
+      <state_interface name="position"/>
+      <state_interface name="velocity"/>
+    </joint>
+    <joint name="joint_2">
+      <command_interface name="position">
+        <param name="min">-1.7453</param>
+        <param name="max">1.9199</param>
+      </command_interface>
+      <state_interface name="position"/>
+      <state_interface name="velocity"/>
+    </joint>
+    <joint name="joint_3">
+      <command_interface name="position">
+        <param name="min">-1.0472</param>
+        <param name="max">1.1345</param>
+      </command_interface>
+      <state_interface name="position"/>
+      <state_interface name="velocity"/>
+    </joint>
+    <joint name="joint_4">
+      <command_interface name="position">
+        <param name="min">-3.49</param>
+        <param name="max">3.49</param>
+      </command_interface>
+      <state_interface name="position"/>
+      <state_interface name="velocity"/>
+    </joint>
+    <joint name="joint_5">
+      <command_interface name="position">
+        <param name="min">-2.0944</param>
+        <param name="max">2.0944</param>
+      </command_interface>
+      <state_interface name="position"/>
+      <state_interface name="velocity"/>
+    </joint>
+    <joint name="joint_6">
+      <command_interface name="position">
+        <param name="min">-6.9813</param>
+        <param name="max">6.9813</param>
+      </command_interface>
+      <state_interface name="position"/>
+      <state_interface name="velocity"/>
+    </joint>
+    <!-- Pneumatic gripper. Only the left finger's first joint is a real
+         driver (position command interface); the other 11 finger joints are
+         declared mimic="true" here and carry <mimic> elements in
+         irb140_pneumonic_gripper_finger.xacro, so a single
+         GripperActionController (config/controllers.yaml: gripper_controller)
+         opens/closes both fingers. Mimic joints may only export state
+         interfaces. -->
+    <joint name="pneumatic_gripper_left_link_1_to_link_2">
+      <!-- Software travel limit for the driver joint: -0.0698 ("closed") is
+           deliberately kept 0.02 rad inside the -0.09 mechanical joint limit
+           (see irb140_pneumonic_gripper_finger.xacro) so a closed gripper is
+           resting, not pegged on the hard stop; opening from closed is then
+           a free move the weak position gain can complete without stalling. -->
+      <command_interface name="position">
+        <param name="min">-0.0698</param>
+        <param name="max">0.0</param>
+      </command_interface>
+      <state_interface name="position"/>
+      <state_interface name="velocity"/>
+    </joint>
+    <joint name="pneumatic_gripper_left_link_2_to_link_3" mimic="true">
+      <state_interface name="position"/>
+      <state_interface name="velocity"/>
+    </joint>
+    <joint name="pneumatic_gripper_left_link_3_to_link_4" mimic="true">
+      <state_interface name="position"/>
+      <state_interface name="velocity"/>
+    </joint>
+    <joint name="pneumatic_gripper_left_link_4_to_link_5" mimic="true">
+      <state_interface name="position"/>
+      <state_interface name="velocity"/>
+    </joint>
+    <joint name="pneumatic_gripper_left_link_5_to_link_6" mimic="true">
+      <state_interface name="position"/>
+      <state_interface name="velocity"/>
+    </joint>
+    <joint name="pneumatic_gripper_left_link_6_to_link_7" mimic="true">
+      <state_interface name="position"/>
+      <state_interface name="velocity"/>
+    </joint>
+    <joint name="pneumatic_gripper_right_link_1_to_link_2" mimic="true">
+      <state_interface name="position"/>
+      <state_interface name="velocity"/>
+    </joint>
+    <joint name="pneumatic_gripper_right_link_2_to_link_3" mimic="true">
+      <state_interface name="position"/>
+      <state_interface name="velocity"/>
+    </joint>
+    <joint name="pneumatic_gripper_right_link_3_to_link_4" mimic="true">
+      <state_interface name="position"/>
+      <state_interface name="velocity"/>
+    </joint>
+    <joint name="pneumatic_gripper_right_link_4_to_link_5" mimic="true">
+      <state_interface name="position"/>
+      <state_interface name="velocity"/>
+    </joint>
+    <joint name="pneumatic_gripper_right_link_5_to_link_6" mimic="true">
+      <state_interface name="position"/>
+      <state_interface name="velocity"/>
+    </joint>
+    <joint name="pneumatic_gripper_right_link_6_to_link_7" mimic="true">
+      <state_interface name="position"/>
+      <state_interface name="velocity"/>
+    </joint>
+  </ros2_control>
+  <!-- Brings up a controller_manager inside gz-sim once the entity is spawned.
+       CONTROLLERS_YAML_PATH is a literal token that launch/gazebo.launch.py
+       rewrites to the installed config/controllers.yaml path before the URDF
+       is published (gz_ros2_control does not evaluate $(find pkg) itself when
+       the description is passed through as plain text). -->
+  <gazebo>
+    <plugin filename="gz_ros2_control-system"
+            name="gz_ros2_control::GazeboSimROS2ControlPlugin">
+      <parameters>CONTROLLERS_YAML_PATH</parameters>
+    </plugin>
+  </gazebo>
 </robot>

File: urdf/irb140_pneumonic_gripper.xacro (robot description, xacro)
@@ -2,4 +2,10 @@
 <robot xmlns:xacro="http://www.ros.org/wiki/xacro" name="pneumatic_gripper">
 <xacro:include filename="$(find abb_irb140_description)/urdf/irb140_pneumonic_gripper_finger.xacro"/>
+<!-- Set include_camera:=false at xacro time to drop the wrist RGBD camera. -->
+<xacro:arg name="include_camera" default="true"/>
+<!-- 3D-printed PLA housing: solid PLA is ~1240 kg/m^3; with typical printed
+     wall/infill this shell is roughly half that, so ~650 kg/m^3 over the
+     bounding box gives a realistic ~0.45 kg body. -->
+<xacro:property name="pla_density" value="650.0"/>
 <xacro:macro name="pneumatic_gripper" params="name parent xyz:='0 0 0' rpy:='0 0 0'">
     <!-- Attach the gripper body to the robot flange.
@@ -27,19 +33,100 @@
             </geometry>
         </collision>
-        <inertial>
-            <mass value="1.0"/>
-            <inertia ixx="0.001" ixy="0" ixz="0" iyy="0.001" iyz="0" izz="0.001"/>
-        </inertial>
+        <xacro:solid_box_inertial sx="0.1" sy="0.125" sz="0.062" density="${pla_density}">
+            <origin xyz="0.0165 0 -0.005" rpy="0 0 0"/>
+        </xacro:solid_box_inertial>
     </link>
     <!-- Spawn left and right gripper fingers.
          The offset/rotation for each finger is passed straight into the
-         finger macro's base joint (its <origin> block). -->
+         finger macro's base joint (its <origin> block).
+         The left finger's first joint (${name}_left_link_1_to_link_2) is the
+         single driver: it gets the ros2_control position command interface in
+         irb140.xacro, and the other 11 finger joints mimic it, so one
+         GripperActionController opens/closes both fingers. -->
     <xacro:pneumatic_gripper_finger name="${name}_left" parent="${name}_base_link">
         <origin xyz="0.0 0.046 0.0071" rpy="0.0 0.0 1.57"/>
     </xacro:pneumatic_gripper_finger>
-    <xacro:pneumatic_gripper_finger name="${name}_right" parent="${name}_base_link">
+    <xacro:pneumatic_gripper_finger name="${name}_right" parent="${name}_base_link"
+                                    mimic_master="${name}_left_link_1_to_link_2">
         <origin xyz="-0.008 -0.046 0.0071" rpy="0.0 0.0 -1.57"/>
     </xacro:pneumatic_gripper_finger>
-    <xacro:arg name="include_camera" default="true"/>
+    <!-- ================================================================= -->
+    <!-- Eye-in-hand RGBD camera                                           -->
+    <!-- ================================================================= -->
+    <!-- Link/sensor/topic names are deliberately un-namespaced
+         (depth_camera / rgbd_camera): config/rgbd_bridge.yaml and
+         launch/gazebo.launch.py refer to them by those fixed names. Only one
+         gripper is ever instantiated, so there is no collision. -->
+    <xacro:if value="$(arg include_camera)">
+        <!-- Geometry-less sensor frame: the physical camera is already
+             sculpted into the base_link visual mesh, so this link carries no
+             visual/collision of its own (that would just duplicate the mesh
+             as a second, floating box). It exists purely so the Gazebo
+             rgbd_camera sensor below has a link to attach to, positioned and
+             rotated (local +X is the gz camera view axis) to coincide with
+             the real camera on the mesh, along the gripper's approach
+             direction (+Z of ${name}_base_link). Tune the joint origin below
+             to reframe the grasp view. -->
+        <link name="depth_camera">
+            <inertial>
+                <mass value="0.05"/>
+                <inertia ixx="1e-5" ixy="0" ixz="0" iyy="1e-5" iyz="0" izz="1e-5"/>
+            </inertial>
+        </link>
+        <joint name="${name}_to_depth_camera" type="fixed">
+            <parent link="${name}_base_link"/>
+            <child link="depth_camera"/>
+            <origin xyz="-0.025 0.0 0.3" rpy="3.14159265359 0 0"/>
+        </joint>
+        <!-- Keep depth_camera as its own link/frame in the converted SDF
+             instead of letting urdf2sdf lump it (and the sensor) back into
+             link_6 through the fixed-joint chain. -->
+        <gazebo reference="${name}_to_depth_camera">
+            <preserveFixedJoint>true</preserveFixedJoint>
+            <disableFixedJointLumping>true</disableFixedJointLumping>
+        </gazebo>
+        <!-- Standard ROS optical frame (z forward, x right, y down) relative to
+             the camera body link; camera_info / point clouds are published in
+             this frame. -->
+        <link name="depth_camera_optical"/>
+        <joint name="depth_camera_to_optical" type="fixed">
+            <parent link="depth_camera"/>
+            <child link="depth_camera_optical"/>
+            <origin xyz="0 0 0" rpy="0 -1.57 0"/>
+        </joint>
+        <!-- reference="depth_camera" binds the gz-sim sensor to that link.
+             worlds/robot_lab.world already loads gz-sim-sensors-system. gz
+             publishes /rgbd_camera/{image,depth_image,points,camera_info};
+             those are remapped to RealSense-style ROS 2 names by
+             config/rgbd_bridge.yaml in launch/gazebo.launch.py. -->
+        <gazebo reference="depth_camera">
+            <sensor name="rgbd_camera" type="rgbd_camera">
+                <always_on>1</always_on>
+                <update_rate>30</update_rate>
+                <visualize>true</visualize>
+                <topic>rgbd_camera</topic>
+                <gz_frame_id>depth_camera</gz_frame_id>
+                <camera>
+                    <horizontal_fov>1.3962634</horizontal_fov>
+                    <image>
+                        <width>640</width>
+                        <height>480</height>
+                        <format>R8G8B8</format>
+                    </image>
+                    <clip>
+                        <near>0.1</near>
+                        <far>15</far>
+                    </clip>
+                    <depth_camera>
+                        <clip>
+                            <near>0.1</near>
+                            <far>15</far>
+                        </clip>
+                    </depth_camera>
+                    <optical_frame_id>depth_camera_optical</optical_frame_id>
+                </camera>
+            </sensor>
+        </gazebo>
+    </xacro:if>
 </xacro:macro>
 </robot>
