Commit message: updates

File: urdf/irb140_pneumonic_gripper_finger.xacro (robot description, xacro)
@@ -4,10 +4,37 @@
     <xacro:property name="mesh_scale" value="0.001 0.001 0.001"/>
     <xacro:property name="collision_scale" value="0.025 0.03 0.1"/>
-    <xacro:property name="joint_lower_limit" value="-0.0698"/>
+    <!-- Mechanical hard stop for each finger segment. The GripperActionController
+         is commanded to -0.0698 for "closed" (command_interface min in
+         irb140.xacro), so this limit sits 0.02 rad beyond that: a closed gripper
+         rests short of the stop instead of jamming against it, which is what let
+         a single-shot open stall out from the fully-closed pose. -->
+    <xacro:property name="joint_lower_limit" value="-0.09"/>
+    <!-- Cast silicone rubber (Dragon Skin / Ecoflex class), ~1100 kg/m^3.
+         Raise this if the finger chain jitters in Gazebo; it scales every
+         segment mass and inertia together. -->
+    <xacro:property name="silicone_density" value="1100.0"/>
     <material name="offwhite">
         <color rgba="0.8 0.8 0.8 1"/>
     </material>
-    <!-- Macro for the finger assembly -->
-    <xacro:macro name="pneumatic_gripper_finger" params="name parent *origin">
+    <!-- Solid-box mass + inertia from full box dimensions (sx,sy,sz) and a
+         material density. Inertia is taken about the box centre, so pass the
+         same *origin used for the matching <collision> box. -->
+    <xacro:macro name="solid_box_inertial" params="sx sy sz density *origin">
+        <inertial>
+            <xacro:insert_block name="origin"/>
+            <mass value="${density * sx * sy * sz}"/>
+            <inertia ixx="${density * sx * sy * sz * (sy*sy + sz*sz) / 12.0}" ixy="0.0" ixz="0.0"
+                     iyy="${density * sx * sy * sz * (sx*sx + sz*sz) / 12.0}" iyz="0.0"
+                     izz="${density * sx * sy * sz * (sx*sx + sy*sy) / 12.0}"/>
+        </inertial>
+    </xacro:macro>
+    <!-- Macro for the finger assembly.
+         mimic_master: leave empty on the driver finger, so its own
+         ${name}_link_1_to_link_2 becomes the joint everything else mimics.
+         Set it to that joint's name on the second finger so both fingers
+         follow a single ros2_control command interface. -->
+    <xacro:macro name="pneumatic_gripper_finger" params="name parent mimic_master:='' *origin">
+        <!-- Joint that every non-driver segment of this finger mimics. -->
+        <xacro:property name="_master" value="${mimic_master if mimic_master else name + '_link_1_to_link_2'}"/>
         <link name="${name}_link_1">
             <visual>
@@ -23,4 +50,7 @@
                 </geometry>
             </collision>
+            <xacro:solid_box_inertial sx="0.025" sy="0.03" sz="0.022" density="${silicone_density}">
+                <origin xyz="0 0.005 0.009" rpy="0 0 0"/>
+            </xacro:solid_box_inertial>
         </link>
         <link name="${name}_link_2">
@@ -37,4 +67,7 @@
                 </geometry>
             </collision>
+            <xacro:solid_box_inertial sx="0.025" sy="0.03" sz="0.011" density="${silicone_density}">
+                <origin xyz="0 0 0.025" rpy="0 0 0"/>
+            </xacro:solid_box_inertial>
         </link>
         <link name="${name}_link_3">
@@ -51,4 +84,7 @@
                 </geometry>
             </collision>
+            <xacro:solid_box_inertial sx="0.025" sy="0.03" sz="0.011" density="${silicone_density}">
+                <origin xyz="0 0 0.035" rpy="0 0 0"/>
+            </xacro:solid_box_inertial>
         </link>
         <link name="${name}_link_4">
@@ -65,4 +101,7 @@
                 </geometry>
             </collision>
+            <xacro:solid_box_inertial sx="0.025" sy="0.03" sz="0.011" density="${silicone_density}">
+                <origin xyz="0 0 0.055" rpy="0 0 0"/>
+            </xacro:solid_box_inertial>
         </link>
         <link name="${name}_link_5">
@@ -79,4 +118,7 @@
                 </geometry>
             </collision>
+            <xacro:solid_box_inertial sx="0.025" sy="0.03" sz="0.011" density="${silicone_density}">
+                <origin xyz="0 0 0.065" rpy="0 0 0"/>
+            </xacro:solid_box_inertial>
         </link>
         <link name="${name}_link_6">
@@ -93,4 +135,7 @@
                 </geometry>
             </collision>
+            <xacro:solid_box_inertial sx="0.025" sy="0.03" sz="0.011" density="${silicone_density}">
+                <origin xyz="0 0 0.075" rpy="0 0 0"/>
+            </xacro:solid_box_inertial>
         </link>
         <link name="${name}_link_7">
@@ -107,4 +152,7 @@
                 </geometry>
             </collision>
+            <xacro:solid_box_inertial sx="0.025" sy="0.03" sz="0.011" density="${silicone_density}">
+                <origin xyz="0 0 0.085" rpy="0 0 0"/>
+            </xacro:solid_box_inertial>
         </link>
         <!-- Base to link_1 joint -->
@@ -121,4 +169,8 @@
             <axis xyz="0 1 0"/>
             <limit lower="${joint_lower_limit}" upper="0" effort="10" velocity="1.0"/>
+            <dynamics damping="0.1"/>
+            <xacro:if value="${mimic_master != ''}">
+                <mimic joint="${mimic_master}" multiplier="1.0" offset="0.0"/>
+            </xacro:if>
         </joint>
         <joint name="${name}_link_2_to_link_3" type="revolute">
@@ -128,4 +180,6 @@
             <axis xyz="0 1 0"/>
             <limit lower="${joint_lower_limit}" upper="0" effort="10" velocity="1.0"/>
+            <dynamics damping="0.1"/>
+            <mimic joint="${_master}" multiplier="1.0" offset="0.0"/>
         </joint>
         <joint name="${name}_link_3_to_link_4" type="revolute">
@@ -135,4 +189,6 @@
             <axis xyz="0 1 0"/>
             <limit lower="${joint_lower_limit}" upper="0" effort="10" velocity="1.0"/>
+            <dynamics damping="0.1"/>
+            <mimic joint="${_master}" multiplier="1.0" offset="0.0"/>
         </joint>
         <joint name="${name}_link_4_to_link_5" type="revolute">
@@ -142,4 +198,6 @@
             <axis xyz="0 1 0"/>
             <limit lower="${joint_lower_limit}" upper="0" effort="10" velocity="1.0"/>
+            <dynamics damping="0.1"/>
+            <mimic joint="${_master}" multiplier="1.0" offset="0.0"/>
         </joint>
         <joint name="${name}_link_5_to_link_6" type="revolute">
@@ -149,4 +207,6 @@
             <axis xyz="0 1 0"/>
             <limit lower="${joint_lower_limit}" upper="0" effort="10" velocity="1.0"/>
+            <dynamics damping="0.1"/>
+            <mimic joint="${_master}" multiplier="1.0" offset="0.0"/>
         </joint>
         <joint name="${name}_link_6_to_link_7" type="revolute">
@@ -156,4 +216,6 @@
             <axis xyz="0 1 0"/>
             <limit lower="${joint_lower_limit}" upper="0" effort="10" velocity="1.0"/>
+            <dynamics damping="0.1"/>
+            <mimic joint="${_master}" multiplier="1.0" offset="0.0"/>
         </joint>
     </xacro:macro>

Commit message: updates

File: urdf/irb140.urdf (robot description, URDF)
Before this commit: robot abb_irb140, 27 links, 26 joints
Joints:
- joint depth_camera_to_optical: origin xyz=0 0 0 rpy=0.0 0.0 0 -> xyz=0 0 0 rpy=-1.57079632679 0 -1.57079632679

File: urdf/irb140_pneumonic_gripper.urdf (robot description, URDF)
Before this commit: robot pneumatic_gripper_standalone, 18 links, 17 joints
Joints:
- joint depth_camera_to_optical: origin xyz=0 0 0 rpy=0 1.57 0 -> xyz=0 0 0 rpy=-1.57079632679 0 -1.57079632679
- joint pneumatic_gripper_to_depth_camera: origin xyz=-0.025 0.0 0.3 rpy=3.14159265359 0 0 -> xyz=-0.025 0.0 0.05 rpy=3.14159265359 -1.57079632679 0

File: urdf/irb140_pneumonic_gripper.xacro (robot description, xacro)
@@ -88,10 +88,16 @@
         <!-- Standard ROS optical frame (z forward, x right, y down) relative to
              the camera body link; camera_info / point clouds are published in
-             this frame. -->
+             this frame. depth_camera's own +X is the gz view axis (see the
+             mount joint above), so this applies the standard body->optical
+             fixed rotation (roll -90, yaw -90) to actually get there;
+             identity here would leave depth_camera_optical pointing the same
+             way as depth_camera despite the data being genuinely
+             optical-convention, which is what was skewing the RViz
+             projection. -->
         <link name="depth_camera_optical"/>
         <joint name="depth_camera_to_optical" type="fixed">
             <parent link="depth_camera"/>
             <child link="depth_camera_optical"/>
-            <origin xyz="0 0 0" rpy="0.0 0.0 0"/>
+            <origin xyz="0 0 0" rpy="-1.57079632679 0 -1.57079632679"/>
         </joint>
         <!-- reference="depth_camera" binds the gz-sim sensor to that link.

Commit message: updates

File: urdf/irb140.urdf (robot description, URDF)
Before this commit: robot abb_irb140, 27 links, 26 joints
Links:
- link pneumatic_gripper_base_link: geometry collision mesh filename=package://abb_irb140_description/meshes/abb_irb140_pneumoni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 scale=0.001 0.001 0.001; visual mesh filename=package://abb_irb140_description/meshes/abb_irb140_pneumoni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 scale=0.001 0.001 0.001
- link pneumatic_gripper_left_link_1: geometry collision mesh filename=package://abb_irb140_description/meshes/abb_irb140_pneumoni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 scale=0.001 0.001 0.001; visual mesh filename=package://abb_irb140_description/meshes/abb_irb140_pneumoni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 scale=0.001 0.001 0.001
- link pneumatic_gripper_left_link_2: geometry collision mesh filename=package://abb_irb140_description/meshes/abb_irb140_pneumoni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 scale=0.001 0.001 0.001; visual mesh filename=package://abb_irb140_description/meshes/abb_irb140_pneumoni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 scale=0.001 0.001 0.001
- link pneumatic_gripper_left_link_3: geometry collision mesh filename=package://abb_irb140_description/meshes/abb_irb140_pneumoni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 scale=0.001 0.001 0.001; visual mesh filename=package://abb_irb140_description/meshes/abb_irb140_pneumoni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 scale=0.001 0.001 0.001
- link pneumatic_gripper_left_link_4: geometry collision mesh filename=package://abb_irb140_description/meshes/abb_irb140_pneumoni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 scale=0.001 0.001 0.001; visual mesh filename=package://abb_irb140_description/meshes/abb_irb140_pneumoni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 scale=0.001 0.001 0.001
- link pneumatic_gripper_left_link_5: geometry collision mesh filename=package://abb_irb140_description/meshes/abb_irb140_pneumoni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 scale=0.001 0.001 0.001; visual mesh filename=package://abb_irb140_description/meshes/abb_irb140_pneumoni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 scale=0.001 0.001 0.001
- link pneumatic_gripper_left_link_6: geometry collision mesh filename=package://abb_irb140_description/meshes/abb_irb140_pneumoni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 scale=0.001 0.001 0.001; visual mesh filename=package://abb_irb140_description/meshes/abb_irb140_pneumoni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 scale=0.001 0.001 0.001
- link pneumatic_gripper_left_link_7: geometry collision mesh filename=package://abb_irb140_description/meshes/abb_irb140_pneumoni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 scale=0.001 0.001 0.001; visual mesh filename=package://abb_irb140_description/meshes/abb_irb140_pneumoni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 scale=0.001 0.001 0.001
- link pneumatic_gripper_right_link_1: geometry collision mesh filename=package://abb_irb140_description/meshes/abb_irb140_pneumoni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 scale=0.001 0.001 0.001; visual mesh filename=package://abb_irb140_description/meshes/abb_irb140_pneumoni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 scale=0.001 0.001 0.001
- link pneumatic_gripper_right_link_2: geometry collision mesh filename=package://abb_irb140_description/meshes/abb_irb140_pneumoni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 scale=0.001 0.001 0.001; visual mesh filename=package://abb_irb140_description/meshes/abb_irb140_pneumoni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 scale=0.001 0.001 0.001
- link pneumatic_gripper_right_link_3: geometry collision mesh filename=package://abb_irb140_description/meshes/abb_irb140_pneumoni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 scale=0.001 0.001 0.001; visual mesh filename=package://abb_irb140_description/meshes/abb_irb140_pneumoni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 scale=0.001 0.001 0.001
- link pneumatic_gripper_right_link_4: geometry collision mesh filename=package://abb_irb140_description/meshes/abb_irb140_pneumoni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 scale=0.001 0.001 0.001; visual mesh filename=package://abb_irb140_description/meshes/abb_irb140_pneumoni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 scale=0.001 0.001 0.001
- link pneumatic_gripper_right_link_5: geometry collision mesh filename=package://abb_irb140_description/meshes/abb_irb140_pneumoni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 scale=0.001 0.001 0.001; visual mesh filename=package://abb_irb140_description/meshes/abb_irb140_pneumoni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 scale=0.001 0.001 0.001
- link pneumatic_gripper_right_link_6: geometry collision mesh filename=package://abb_irb140_description/meshes/abb_irb140_pneumoni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 scale=0.001 0.001 0.001; visual mesh filename=package://abb_irb140_description/meshes/abb_irb140_pneumoni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 scale=0.001 0.001 0.001
- link pneumatic_gripper_right_link_7: geometry collision mesh filename=package://abb_irb140_description/meshes/abb_irb140_pneumoni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 scale=0.001 0.001 0.001; visual mesh filename=package://abb_irb140_description/meshes/abb_irb140_pneumoni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 scale=0.001 0.001 0.001

File: urdf/irb140_pneumonic_gripper.urdf (robot description, URDF)
Before this commit: robot pneumatic_gripper_standalone, 18 links, 17 joints
Links:
- link pneumatic_gripper_base_link: geometry collision mesh filename=package://abb_irb140_description/meshes/abb_irb140_pneumoni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 scale=0.001 0.001 0.001; visual mesh filename=package://abb_irb140_description/meshes/abb_irb140_pneumoni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 scale=0.001 0.001 0.001

File: urdf/irb140_pneumonic_gripper.xacro (robot description, xacro)
@@ -28,7 +28,7 @@
         </visual>
         <collision>
-            <origin xyz="0.0165 0 -0.005" rpy="0 0 0"/>
+            <origin rpy="0 0 0" xyz="0 0 -0.03105"/>
             <geometry>
-                <box size="0.1 0.125 0.062"/>
+                <mesh filename="package://abb_irb140_description/meshes/abb_irb140_pneumonic_end_effector/visual/ABBIRB140_EndEffector.stl" scale="0.001 0.001 0.001"/>
             </geometry>
         </collision>

File: urdf/irb140_pneumonic_gripper_finger.xacro (robot description, xacro)
@@ -55,7 +55,6 @@
             </visual>
             <collision>
-                <origin xyz="0 0.005 0.009" rpy="0 0 0"/>
-                <geometry>
-                    <box size="0.025 0.03 0.022"/>
+                <geometry>
+                    <mesh filename="package://abb_irb140_description/meshes/abb_irb140_pneumonic_end_effector/visual/finger_visual/visual/link_1.stl" scale="${mesh_scale}"/>
                 </geometry>
             </collision>
@@ -72,11 +71,10 @@
             </visual>
             <collision>
+                <geometry>
+                    <mesh filename="package://abb_irb140_description/meshes/abb_irb140_pneumonic_end_effector/visual/finger_visual/visual/link_2.stl" scale="${mesh_scale}"/>
+                </geometry>
+            </collision>
+            <xacro:solid_box_inertial sx="0.025" sy="0.03" sz="0.011" density="${silicone_density}">
                 <origin xyz="0 0 0.025" rpy="0 0 0"/>
-                <geometry>
-                    <box size="0.025 0.03 0.011"/>
-                </geometry>
-            </collision>
-            <xacro:solid_box_inertial sx="0.025" sy="0.03" sz="0.011" density="${silicone_density}">
-                <origin xyz="0 0 0.025" rpy="0 0 0"/>
             </xacro:solid_box_inertial>
         </link>
@@ -89,11 +87,10 @@
             </visual>
             <collision>
+                <geometry>
+                    <mesh filename="package://abb_irb140_description/meshes/abb_irb140_pneumonic_end_effector/visual/finger_visual/visual/link_3.stl" scale="${mesh_scale}"/>
+                </geometry>
+            </collision>
+            <xacro:solid_box_inertial sx="0.025" sy="0.03" sz="0.011" density="${silicone_density}">
                 <origin xyz="0 0 0.035" rpy="0 0 0"/>
-                <geometry>
-                    <box size="0.025 0.03 0.011"/>
-                </geometry>
-            </collision>
-            <xacro:solid_box_inertial sx="0.025" sy="0.03" sz="0.011" density="${silicone_density}">
-                <origin xyz="0 0 0.035" rpy="0 0 0"/>
             </xacro:solid_box_inertial>
         </link>
@@ -106,11 +103,10 @@
             </visual>
             <collision>
+                <geometry>
+                    <mesh filename="package://abb_irb140_description/meshes/abb_irb140_pneumonic_end_effector/visual/finger_visual/visual/link_4.stl" scale="${mesh_scale}"/>
+                </geometry>
+            </collision>
+            <xacro:solid_box_inertial sx="0.025" sy="0.03" sz="0.011" density="${silicone_density}">
                 <origin xyz="0 0 0.055" rpy="0 0 0"/>
-                <geometry>
-                    <box size="0.025 0.03 0.011"/>
-                </geometry>
-            </collision>
-            <xacro:solid_box_inertial sx="0.025" sy="0.03" sz="0.011" density="${silicone_density}">
-                <origin xyz="0 0 0.055" rpy="0 0 0"/>
             </xacro:solid_box_inertial>
         </link>
@@ -123,11 +119,10 @@
             </visual>
             <collision>
+                <geometry>
+                    <mesh filename="package://abb_irb140_description/meshes/abb_irb140_pneumonic_end_effector/visual/finger_visual/visual/link_5.stl" scale="${mesh_scale}"/>
+                </geometry>
+            </collision>
+            <xacro:solid_box_inertial sx="0.025" sy="0.03" sz="0.011" density="${silicone_density}">
                 <origin xyz="0 0 0.065" rpy="0 0 0"/>
-                <geometry>
-                    <box size="0.025 0.03 0.011"/>
-                </geometry>
-            </collision>
-            <xacro:solid_box_inertial sx="0.025" sy="0.03" sz="0.011" density="${silicone_density}">
-                <origin xyz="0 0 0.065" rpy="0 0 0"/>
             </xacro:solid_box_inertial>
         </link>
@@ -140,11 +135,10 @@
             </visual>
             <collision>
+                <geometry>
+                    <mesh filename="package://abb_irb140_description/meshes/abb_irb140_pneumonic_end_effector/visual/finger_visual/visual/link_6.stl" scale="${mesh_scale}"/>
+                </geometry>
+            </collision>
+            <xacro:solid_box_inertial sx="0.025" sy="0.03" sz="0.011" density="${silicone_density}">
                 <origin xyz="0 0 0.075" rpy="0 0 0"/>
-                <geometry>
-                    <box size="0.025 0.03 0.011"/>
-                </geometry>
-            </collision>
-            <xacro:solid_box_inertial sx="0.025" sy="0.03" sz="0.011" density="${silicone_density}">
-                <origin xyz="0 0 0.075" rpy="0 0 0"/>
             </xacro:solid_box_inertial>
         </link>
@@ -157,7 +151,6 @@
             </visual>
             <collision>
-                <origin xyz="0 0 0.085" rpy="0 0 0"/>
-                <geometry>
-                    <box size="0.025 0.03 0.011"/>
+                <geometry>
+                    <mesh filename="package://abb_irb140_description/meshes/abb_irb140_pneumonic_end_effector/visual/finger_visual/visual/link_7.stl" scale="${mesh_scale}"/>
                 </geometry>
             </collision>
