Commit message: tidy up - fixing naming mistakes and removing olds packages

File: urdf/irb140.urdf (robot description, URDF)
Before this commit: robot abb_irb140, 27 links, 26 joints
Links:
- link pneumatic_gripper_base_link: geometry collision mesh filename=package://abb_irb140_description/meshes/abb_irb140_pneumati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 scale=0.001 0.001 0.001; visual mesh filename=package://abb_irb140_description/meshes/abb_irb140_pneumati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 scale=0.001 0.001 0.001
- link pneumatic_gripper_left_link_1: geometry collision mesh filename=package://abb_irb140_description/meshes/abb_irb140_pneumati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 scale=0.001 0.001 0.001; visual mesh filename=package://abb_irb140_description/meshes/abb_irb140_pneumati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 scale=0.001 0.001 0.001
- link pneumatic_gripper_left_link_2: geometry collision mesh filename=package://abb_irb140_description/meshes/abb_irb140_pneumati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 scale=0.001 0.001 0.001; visual mesh filename=package://abb_irb140_description/meshes/abb_irb140_pneumati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 scale=0.001 0.001 0.001
- link pneumatic_gripper_left_link_3: geometry collision mesh filename=package://abb_irb140_description/meshes/abb_irb140_pneumati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 scale=0.001 0.001 0.001; visual mesh filename=package://abb_irb140_description/meshes/abb_irb140_pneumati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 scale=0.001 0.001 0.001
- link pneumatic_gripper_left_link_4: geometry collision mesh filename=package://abb_irb140_description/meshes/abb_irb140_pneumati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 scale=0.001 0.001 0.001; visual mesh filename=package://abb_irb140_description/meshes/abb_irb140_pneumati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 scale=0.001 0.001 0.001
- link pneumatic_gripper_left_link_5: geometry collision mesh filename=package://abb_irb140_description/meshes/abb_irb140_pneumati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 scale=0.001 0.001 0.001; visual mesh filename=package://abb_irb140_description/meshes/abb_irb140_pneumati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 scale=0.001 0.001 0.001
- link pneumatic_gripper_left_link_6: geometry collision mesh filename=package://abb_irb140_description/meshes/abb_irb140_pneumati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 scale=0.001 0.001 0.001; visual mesh filename=package://abb_irb140_description/meshes/abb_irb140_pneumati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 scale=0.001 0.001 0.001
- link pneumatic_gripper_left_link_7: geometry collision mesh filename=package://abb_irb140_description/meshes/abb_irb140_pneumati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 scale=0.001 0.001 0.001; visual mesh filename=package://abb_irb140_description/meshes/abb_irb140_pneumati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 scale=0.001 0.001 0.001
- link pneumatic_gripper_right_link_1: geometry collision mesh filename=package://abb_irb140_description/meshes/abb_irb140_pneumati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 scale=0.001 0.001 0.001; visual mesh filename=package://abb_irb140_description/meshes/abb_irb140_pneumati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 scale=0.001 0.001 0.001
- link pneumatic_gripper_right_link_2: geometry collision mesh filename=package://abb_irb140_description/meshes/abb_irb140_pneumati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 scale=0.001 0.001 0.001; visual mesh filename=package://abb_irb140_description/meshes/abb_irb140_pneumati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 scale=0.001 0.001 0.001
- link pneumatic_gripper_right_link_3: geometry collision mesh filename=package://abb_irb140_description/meshes/abb_irb140_pneumati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 scale=0.001 0.001 0.001; visual mesh filename=package://abb_irb140_description/meshes/abb_irb140_pneumati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 scale=0.001 0.001 0.001
- link pneumatic_gripper_right_link_4: geometry collision mesh filename=package://abb_irb140_description/meshes/abb_irb140_pneumati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 scale=0.001 0.001 0.001; visual mesh filename=package://abb_irb140_description/meshes/abb_irb140_pneumati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 scale=0.001 0.001 0.001
- link pneumatic_gripper_right_link_5: geometry collision mesh filename=package://abb_irb140_description/meshes/abb_irb140_pneumati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 scale=0.001 0.001 0.001; visual mesh filename=package://abb_irb140_description/meshes/abb_irb140_pneumati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 scale=0.001 0.001 0.001
- link pneumatic_gripper_right_link_6: geometry collision mesh filename=package://abb_irb140_description/meshes/abb_irb140_pneumati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 scale=0.001 0.001 0.001; visual mesh filename=package://abb_irb140_description/meshes/abb_irb140_pneumati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 scale=0.001 0.001 0.001
- link pneumatic_gripper_right_link_7: geometry collision mesh filename=package://abb_irb140_description/meshes/abb_irb140_pneumati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 scale=0.001 0.001 0.001; visual mesh filename=package://abb_irb140_description/meshes/abb_irb140_pneumati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 scale=0.001 0.001 0.001

File: urdf/irb140.xacro (robot description, xacro)
@@ -1,5 +1,5 @@
 <?xml version="1.0" ?>
 <robot xmlns:xacro="https://www.ros.org/wiki/xacro" name="abb_irb140">
-  <xacro:include filename="$(find abb_irb140_description)/urdf/irb140_pneumonic_gripper.xacro"/>
+  <xacro:include filename="$(find abb_irb140_description)/urdf/irb140_pneumatic_gripper.xacro"/>
   <!-- Path to the ros2_control controller config, consumed by the
        gz_ros2_control plugin's <parameters> tag below. launch/gazebo.launch.py
@@ -294,5 +294,5 @@
          driver (position command interface); the other 11 finger joints are
          declared mimic="true" here and carry <mimic> elements in
-         irb140_pneumonic_gripper_finger.xacro, so a single
+         irb140_pneumatic_gripper_finger.xacro, so a single
          GripperActionController (config/controllers.yaml: gripper_controller)
          opens/closes both fingers. Mimic joints may only export state
@@ -301,5 +301,5 @@
       <!-- Software travel limit for the driver joint: -0.0698 ("closed") is
            deliberately kept 0.02 rad inside the -0.09 mechanical joint limit
-           (see irb140_pneumonic_gripper_finger.xacro) so a closed gripper is
+           (see irb140_pneumatic_gripper_finger.xacro) so a closed gripper is
            resting, not pegged on the hard stop; opening from closed is then
            a free move the weak position gain can complete without stalling. -->

File: urdf/irb140_pneumatic_gripper.xacro (robot description, xacro)
@@ -1,5 +1,5 @@
 <?xml version="1.0" encoding="UTF-8"?>
 <robot xmlns:xacro="http://www.ros.org/wiki/xacro" name="pneumatic_gripper">
-<xacro:include filename="$(find abb_irb140_description)/urdf/irb140_pneumonic_gripper_finger.xacro"/>
+<xacro:include filename="$(find abb_irb140_description)/urdf/irb140_pneumatic_gripper_finger.xacro"/>
 <!-- Set include_camera:=false at xacro time to drop the wrist RGBD camera. -->
 <xacro:arg name="include_camera" default="true"/>
@@ -21,5 +21,5 @@
             <origin xyz="0 0 -0.03105" rpy="0 0 0"/>
             <geometry>
-                <mesh filename="package://abb_irb140_description/meshes/abb_irb140_pneumonic_end_effector/visual/ABBIRB140_EndEffector.stl" scale="0.001 0.001 0.001"/>
+                <mesh filename="package://abb_irb140_description/meshes/abb_irb140_pneumatic_end_effector/visual/ABBIRB140_EndEffector.stl" scale="0.001 0.001 0.001"/>
             </geometry>
             <material name="plastic">
@@ -30,5 +30,5 @@
             <origin rpy="0 0 0" xyz="0 0 -0.03105"/>
             <geometry>
-                <mesh filename="package://abb_irb140_description/meshes/abb_irb140_pneumonic_end_effector/visual/ABBIRB140_EndEffector.stl" scale="0.001 0.001 0.001"/>
+                <mesh filename="package://abb_irb140_description/meshes/abb_irb140_pneumatic_end_effector/visual/ABBIRB140_EndEffector.stl" scale="0.001 0.001 0.001"/>
             </geometry>
         </collision>

File: urdf/irb140_pneumatic_gripper_finger.xacro (robot description, xacro)
@@ -50,11 +50,11 @@
             <visual>
                 <geometry>
-                    <mesh filename="package://abb_irb140_description/meshes/abb_irb140_pneumonic_end_effector/visual/finger_visual/visual/link_1.stl" scale="${mesh_scale}"/>
-                </geometry>
-                <material name="offwhite"/>
-            </visual>
-            <collision>
-                <geometry>
-                    <mesh filename="package://abb_irb140_description/meshes/abb_irb140_pneumonic_end_effector/visual/finger_visual/visual/link_1.stl" scale="${mesh_scale}"/>
+                    <mesh filename="package://abb_irb140_description/meshes/abb_irb140_pneumatic_end_effector/visual/finger_visual/visual/link_1.stl" scale="${mesh_scale}"/>
+                </geometry>
+                <material name="offwhite"/>
+            </visual>
+            <collision>
+                <geometry>
+                    <mesh filename="package://abb_irb140_description/meshes/abb_irb140_pneumatic_end_effector/visual/finger_visual/visual/link_1.stl" scale="${mesh_scale}"/>
                 </geometry>
             </collision>
@@ -66,11 +66,11 @@
             <visual>
                 <geometry>
-                    <mesh filename="package://abb_irb140_description/meshes/abb_irb140_pneumonic_end_effector/visual/finger_visual/visual/link_2.stl" scale="${mesh_scale}"/>
-                </geometry>
-                <material name="offwhite"/>
-            </visual>
-            <collision>
-                <geometry>
-                    <mesh filename="package://abb_irb140_description/meshes/abb_irb140_pneumonic_end_effector/visual/finger_visual/visual/link_2.stl" scale="${mesh_scale}"/>
+                    <mesh filename="package://abb_irb140_description/meshes/abb_irb140_pneumatic_end_effector/visual/finger_visual/visual/link_2.stl" scale="${mesh_scale}"/>
+                </geometry>
+                <material name="offwhite"/>
+            </visual>
+            <collision>
+                <geometry>
+                    <mesh filename="package://abb_irb140_description/meshes/abb_irb140_pneumatic_end_effector/visual/finger_visual/visual/link_2.stl" scale="${mesh_scale}"/>
                 </geometry>
             </collision>
@@ -82,11 +82,11 @@
             <visual>
                 <geometry>
-                    <mesh filename="package://abb_irb140_description/meshes/abb_irb140_pneumonic_end_effector/visual/finger_visual/visual/link_3.stl" scale="${mesh_scale}"/>
-                </geometry>
-                <material name="offwhite"/>
-            </visual>
-            <collision>
-                <geometry>
-                    <mesh filename="package://abb_irb140_description/meshes/abb_irb140_pneumonic_end_effector/visual/finger_visual/visual/link_3.stl" scale="${mesh_scale}"/>
+                    <mesh filename="package://abb_irb140_description/meshes/abb_irb140_pneumatic_end_effector/visual/finger_visual/visual/link_3.stl" scale="${mesh_scale}"/>
+                </geometry>
+                <material name="offwhite"/>
+            </visual>
+            <collision>
+                <geometry>
+                    <mesh filename="package://abb_irb140_description/meshes/abb_irb140_pneumatic_end_effector/visual/finger_visual/visual/link_3.stl" scale="${mesh_scale}"/>
                 </geometry>
             </collision>
@@ -98,11 +98,11 @@
             <visual>
                 <geometry>
-                    <mesh filename="package://abb_irb140_description/meshes/abb_irb140_pneumonic_end_effector/visual/finger_visual/visual/link_4.stl" scale="${mesh_scale}"/>
-                </geometry>
-                <material name="offwhite"/>
-            </visual>
-            <collision>
-                <geometry>
-                    <mesh filename="package://abb_irb140_description/meshes/abb_irb140_pneumonic_end_effector/visual/finger_visual/visual/link_4.stl" scale="${mesh_scale}"/>
+                    <mesh filename="package://abb_irb140_description/meshes/abb_irb140_pneumatic_end_effector/visual/finger_visual/visual/link_4.stl" scale="${mesh_scale}"/>
+                </geometry>
+                <material name="offwhite"/>
+            </visual>
+            <collision>
+                <geometry>
+                    <mesh filename="package://abb_irb140_description/meshes/abb_irb140_pneumatic_end_effector/visual/finger_visual/visual/link_4.stl" scale="${mesh_scale}"/>
                 </geometry>
             </collision>
@@ -114,11 +114,11 @@
             <visual>
                 <geometry>
-                    <mesh filename="package://abb_irb140_description/meshes/abb_irb140_pneumonic_end_effector/visual/finger_visual/visual/link_5.stl" scale="${mesh_scale}"/>
-                </geometry>
-                <material name="offwhite"/>
-            </visual>
-            <collision>
-                <geometry>
-                    <mesh filename="package://abb_irb140_description/meshes/abb_irb140_pneumonic_end_effector/visual/finger_visual/visual/link_5.stl" scale="${mesh_scale}"/>
+                    <mesh filename="package://abb_irb140_description/meshes/abb_irb140_pneumatic_end_effector/visual/finger_visual/visual/link_5.stl" scale="${mesh_scale}"/>
+                </geometry>
+                <material name="offwhite"/>
+            </visual>
+            <collision>
+                <geometry>
+                    <mesh filename="package://abb_irb140_description/meshes/abb_irb140_pneumatic_end_effector/visual/finger_visual/visual/link_5.stl" scale="${mesh_scale}"/>
                 </geometry>
             </collision>
@@ -130,11 +130,11 @@
             <visual>
                 <geometry>
-                    <mesh filename="package://abb_irb140_description/meshes/abb_irb140_pneumonic_end_effector/visual/finger_visual/visual/link_6.stl" scale="${mesh_scale}"/>
-                </geometry>
-                <material name="offwhite"/>
-            </visual>
-            <collision>
-                <geometry>
-                    <mesh filename="package://abb_irb140_description/meshes/abb_irb140_pneumonic_end_effector/visual/finger_visual/visual/link_6.stl" scale="${mesh_scale}"/>
+                    <mesh filename="package://abb_irb140_description/meshes/abb_irb140_pneumatic_end_effector/visual/finger_visual/visual/link_6.stl" scale="${mesh_scale}"/>
+                </geometry>
+                <material name="offwhite"/>
+            </visual>
+            <collision>
+                <geometry>
+                    <mesh filename="package://abb_irb140_description/meshes/abb_irb140_pneumatic_end_effector/visual/finger_visual/visual/link_6.stl" scale="${mesh_scale}"/>
                 </geometry>
             </collision>
@@ -146,11 +146,11 @@
             <visual>
                 <geometry>
-                    <mesh filename="package://abb_irb140_description/meshes/abb_irb140_pneumonic_end_effector/visual/finger_visual/visual/link_7.stl" scale="${mesh_scale}"/>
-                </geometry>
-                <material name="offwhite"/>
-            </visual>
-            <collision>
-                <geometry>
-                    <mesh filename="package://abb_irb140_description/meshes/abb_irb140_pneumonic_end_effector/visual/finger_visual/visual/link_7.stl" scale="${mesh_scale}"/>
+                    <mesh filename="package://abb_irb140_description/meshes/abb_irb140_pneumatic_end_effector/visual/finger_visual/visual/link_7.stl" scale="${mesh_scale}"/>
+                </geometry>
+                <material name="offwhite"/>
+            </visual>
+            <collision>
+                <geometry>
+                    <mesh filename="package://abb_irb140_description/meshes/abb_irb140_pneumatic_end_effector/visual/finger_visual/visual/link_7.stl" scale="${mesh_scale}"/>
                 </geometry>
             </collision>
